File: SafetySupply/SafetySupply.sch (KiCad schematic (older format))
At the start: 34 parts

Commit message: Added horn protection diode. Added some footprints to the elements.
Parts:
- removed D?: LED, Diode_SMD:D_0805_2012Metric, symbol Device:LED
- removed D?: DIODE, symbol pspice:DIODE
- added D? (x2): D_ALT, Diode_SMD:D_MiniMELF, symbol Device:D_ALT
- added D?: LED_ALT, LED_SMD:LED_0805_2012Metric, symbol Device:LED_ALT
- C? (x3): footprint (none) -> Capacitor_SMD:C_0603_1608Metric
- C?: footprint (none) -> Capacitor_SMD:C_0805_2012Metric
Connections:
- wire segments 73 -> 75
Other:
- moved on the sheet: J?
Changed lines of the file:
@@
 F 0 "C?" H 1750 2350 50  0000 L CNN
 F 1 "100n" H 1750 2250 50  0000 L CNN
-F 2 "" H 2088 2150 50  0001 C CNN
+F 2 "Capacitor_SMD:C_0603_1608Metric" H 2088 2150 50  0001 C CNN
 F 3 "~" H 2050 2300 50  0001 C CNN
 	1    2050 2300
@@
 	2250 2450 2050 2450
 $Comp
-L power:+12V #PWR?
+L power:+12V #PWR0101
 U 1 1 5C5F7175
-P 3150 1700
-F 0 "#PWR?" H 3150 1550 50  0001 C CNN
-F 1 "+12V" H 3165 1873 50  0000 C CNN
-F 2 "" H 3150 1700 50  0001 C CNN
-F 3 "" H 3150 1700 50  0001 C CNN
-	1    3150 1700
+P 3150 1750
+F 0 "#PWR0101" H 3150 1600 50  0001 C CNN
+F 1 "+12V" H 3165 1923 50  0000 C CNN
+F 2 "" H 3150 1750 50  0001 C CNN
+F 3 "" H 3150 1750 50  0001 C CNN
+	1    3150 1750
 	1    0    0    -1
 $EndComp
@@
 	1650 2150 1700 2150
 $Comp
-L power:+12V #PWR?
+L power:+12V #PWR0102
 U 1 1 5C6049A1
 P 4450 3200
-F 0 "#PWR?" H 4450 3050 50  0001 C CNN
+F 0 "#PWR0102" H 4450 3050 50  0001 C CNN
 F 1 "+12V" H 4465 3373 50  0000 C CNN
 F 2 "" H 4450 3200 50  0001 C CNN
@@
 $EndComp
 $Comp
-L power:GND #PWR?
+L power:GND #PWR0103
 U 1 1 5C605EC8
 P 4450 4100
-F 0 "#PWR?" H 4450 3850 50  0001 C CNN
+F 0 "#PWR0103" H 4450 3850 50  0001 C CNN
 F 1 "GND" H 4455 3927 50  0000 C CNN
 F 2 "" H 4450 4100 50  0001 C CNN
@@
 	4450 3200 4450 3350
 $Comp
-L Device:LED D?
-U 1 1 5C60CC3E
-P 4450 3800
-F 0 "D?" V 4488 3683 50  0000 R CNN
-F 1 "LED" V 4397 3683 50  0000 R CNN
-F 2 "Diode_SMD:D_0805_2012Metric" H 4450 3800 50  0001 C CNN
-F 3 "~" H 4450 3800 50  0001 C CNN
-	1    4450 3800
-	0    -1   -1   0
-$EndComp
-$Comp
 L Connector:Screw_Terminal_01x02 J?
 U 1 1 5C6116CB
-P 8450 1750
-F 0 "J?" H 8400 1850 50  0000 C CNN
-F 1 "Screw_Terminal_01x02" H 8370 1876 50  0001 C CNN
-F 2 "" H 8450 1750 50  0001 C CNN
-F 3 "~" H 8450 1750 50  0001 C CNN
-	1    8450 1750
+P 8700 1750
+F 0 "J?" H 8650 1850 50  0000 C CNN
+F 1 "Screw_Terminal_01x02" H 8620 1876 50  0001 C CNN
+F 2 "" H 8700 1750 50  0001 C CNN
+F 3 "~" H 8700 1750 50  0001 C CNN
+	1    8700 1750
 	1    0    0    -1
 $EndComp
@@
 $EndComp
 $Comp
-L power:GND #PWR?
+L power:GND #PWR0104
 U 1 1 5C61B126
-P 8250 2050
-F 0 "#PWR?" H 8250 1800 50  0001 C CNN
-F 1 "GND" H 8255 1877 50  0000 C CNN
-F 2 "" H 8250 2050 50  0001 C CNN
-F 3 "" H 8250 2050 50  0001 C CNN
-	1    8250 2050
-	1    0    0    -1
-$EndComp
-$Comp
-L power:+12V #PWR?
+P 8500 2050
+F 0 "#PWR0104" H 8500 1800 50  0001 C CNN
+F 1 "GND" H 8505 1877 50  0000 C CNN
+F 2 "" H 8500 2050 50  0001 C CNN
+F 3 "" H 8500 2050 50  0001 C CNN
+	1    8500 2050
+	1    0    0    -1
+$EndComp
+$Comp
+L power:+12V #PWR0105
 U 1 1 5C61F508
 P 6150 1600
-F 0 "#PWR?" H 6150 1450 50  0001 C CNN
+F 0 "#PWR0105" H 6150 1450 50  0001 C CNN
 F 1 "+12V" H 6165 1773 50  0000 C CNN
 F 2 "" H 6150 1600 50  0001 C CNN
@@
 	6150 2150 6350 2150
 Connection ~ 6150 1750
-$Comp
-L pspice:DIODE D?
-U 1 1 5C623BB2
-P 6650 2550
-F 0 "D?" H 6700 2750 50  0000 C CNN
-F 1 "DIODE" H 6650 2724 50  0001 C CNN
-F 2 "" H 6650 2550 50  0001 C CNN
-F 3 "~" H 6650 2550 50  0001 C CNN
-	1    6650 2550
-	-1   0    0    1
-$EndComp
-Wire Wire Line
-	6450 2550 6150 2550
 Wire Wire Line
 	6150 2550 6150 2150
 Connection ~ 6150 2150
-Wire Wire Line
-	6850 2550 7050 2550
 Wire Wire Line
 	7050 2550 7050 2150
@@
 $EndComp
 $Comp
-L power:GND #PWR?
+L power:GND #PWR0106
 U 1 1 5C627165
 P 7050 2650
-F 0 "#PWR?" H 7050 2400 50  0001 C CNN
+F 0 "#PWR0106" H 7050 2400 50  0001 C CNN
 F 1 "GND" H 7055 2477 50  0000 C CNN
 F 2 "" H 7050 2650 50  0001 C CNN
@@
 $EndComp
 Connection ~ 7050 2550
-Text Notes 8600 1850 0    50   ~ 0
+Text Notes 8900 1850 0    50   ~ 0
 Złącze na klakson
 Text Notes 7400 2650 0    50   ~ 0
@@
 F 0 "C?" H 1750 3700 50  0000 L CNN
 F 1 "100n" H 1750 3600 50  0000 L CNN
-F 2 "" H 2088 3500 50  0001 C CNN
+F 2 "Capacitor_SMD:C_0603_1608Metric" H 2088 3500 50  0001 C CNN
 F 3 "~" H 2050 3650 50  0001 C CNN
 	1    2050 3650
@@
 F 0 "C?" H 1750 5050 50  0000 L CNN
 F 1 "100n" H 1750 4950 50  0000 L CNN
-F 2 "" H 2088 4850 50  0001 C CNN
+F 2 "Capacitor_SMD:C_0603_1608Metric" H 2088 4850 50  0001 C CNN
 F 3 "~" H 2050 5000 50  0001 C CNN
 	1    2050 5000
@@
 Connection ~ 1650 4850
 $Comp
-L power:GND #PWR?
+L power:GND #PWR0107
 U 1 1 5C64DF68
 P 3250 5700
-F 0 "#PWR?" H 3250 5450 50  0001 C CNN
+F 0 "#PWR0107" H 3250 5450 50  0001 C CNN
 F 1 "GND" H 3255 5527 50  0000 C CNN
 F 2 "" H 3250 5700 50  0001 C CNN
@@
 	1    0    0    -1
 $EndComp
-Wire Wire Line
-	3150 1700 3150 1800
 Wire Wire Line
 	3150 1800 2950 1800
@@
 $EndComp
 $Comp
-L power:GND #PWR?
+L power:GND #PWR0108
 U 1 1 5C65FD72
 P 6550 4000
-F 0 "#PWR?" H 6550 3750 50  0001 C CNN
+F 0 "#PWR0108" H 6550 3750 50  0001 C CNN
 F 1 "GND" H 6555 3827 50  0000 C CNN
 F 2 "" H 6550 4000 50  0001 C CNN
@@
 Wyjście napięcia baterii
 $Comp
-L power:+12V #PWR?
+L power:+12V #PWR0109
 U 1 1 5C660F53
 P 6550 3900
-F 0 "#PWR?" H 6550 3750 50  0001 C CNN
+F 0 "#PWR0109" H 6550 3750 50  0001 C CNN
 F 1 "+12V" H 6565 4073 50  0000 C CNN
 F 2 "" H 6550 3900 50  0001 C CNN
@@
 $EndComp
 $Comp
-L power:+12V #PWR?
+L power:+12V #PWR0110
 U 1 1 5C664AD5
 P 3850 1750
-F 0 "#PWR?" H 3850 1600 50  0001 C CNN
+F 0 "#PWR0110" H 3850 1600 50  0001 C CNN
 F 1 "+12V" H 3865 1923 50  0000 C CNN
 F 2 "" H 3850 1750 50  0001 C CNN
@@
 $EndComp
 $Comp
-L power:GND #PWR?
+L power:GND #PWR0111
 U 1 1 5C664B16
 P 3850 2050
-F 0 "#PWR?" H 3850 1800 50  0001 C CNN
+F 0 "#PWR0111" H 3850 1800 50  0001 C CNN
 F 1 "GND" H 3855 1877 50  0000 C CNN
 F 2 "" H 3850 2050 50  0001 C CNN
@@
 F 0 "C?" H 4415 1946 50  0000 L CNN
 F 1 "100n" H 4415 1855 50  0000 L CNN
-F 2 "" H 4338 1750 50  0001 C CNN
+F 2 "Capacitor_SMD:C_0805_2012Metric" H 4338 1750 50  0001 C CNN
 F 3 "~" H 4300 1900 50  0001 C CNN
 	1    4300 1900
@@
 	6950 1750 7200 1750
 Wire Wire Line
-	8250 2050 8250 1850
-Wire Wire Line
-	8250 2050 7950 2050
-Connection ~ 8250 2050
+	8500 2050 8500 1850
+Connection ~ 8500 2050
 Connection ~ 7950 2050
 Connection ~ 7950 1750
-Wire Wire Line
-	7950 1750 8250 1750
 Connection ~ 3250 5550
 Text Notes 3950 1450 0    50   ~ 0
@@
 Text Notes 7300 1500 0    50   ~ 0
 Dodatkowe zabezpieczenia klaksonu
+$Comp
+L Device:D_ALT D?
+U 1 1 5C62AB5D
+P 8200 1900
+F 0 "D?" V 8200 1979 50  0000 L CNN
+F 1 "D_ALT" V 8245 1979 50  0001 L CNN
+F 2 "Diode_SMD:D_MiniMELF" H 8200 1900 50  0001 C CNN
+F 3 "~" H 8200 1900 50  0001 C CNN
+	1    8200 1900
+	0    1    1    0
+$EndComp
+Wire Wire Line
+	7950 1750 8200 1750
+Wire Wire Line
+	7950 2050 8200 2050
+$Comp
+L Device:D_ALT D?
+U 1 1 5C62DCD1
+P 6650 2550
+F 0 "D?" H 6650 2674 50  0000 C CNN
+F 1 "D_ALT" V 6695 2629 50  0001 L CNN
+F 2 "Diode_SMD:D_MiniMELF" H 6650 2550 50  0001 C CNN
+F 3 "~" H 6650 2550 50  0001 C CNN
+	1    6650 2550
+	1    0    0    -1
+$EndComp
+Wire Wire Line
+	6800 2550 7050 2550
+Connection ~ 8200 1750
+Wire Wire Line
+	8200 1750 8500 1750
+Connection ~ 8200 2050
+Wire Wire Line
+	8200 2050 8500 2050
+Wire Wire Line
+	6150 2550 6500 2550
+$Comp
+L Device:LED_ALT D?
+U 1 1 5C638B5A
+P 4450 3800
+F 0 "D?" V 4442 3682 50  0000 R CNN
+F 1 "LED_ALT" V 4397 3682 50  0001 R CNN
+F 2 "LED_SMD:LED_0805_2012Metric" H 4450 3800 50  0001 C CNN
+F 3 "~" H 4450 3800 50  0001 C CNN
+	1    4450 3800
+	0    -1   -1   0
+$EndComp
+Wire Wire Line
+	3150 1750 3150 1800
 $EndSCHEMATC

Commit message: Li-ion polarity protection
commit b1813cd9200a201421d0e06ac9dd889f1f3910dd
Author: Paweł <mackipawel@gmail.com>
Date:   Tue Feb 12 22:32:27 2019 +0100

    Added li-ion polarity protection.
Parts:
- removed C? (x2): 100n, Capacitor_SMD:C_0603_1608Metric, symbol Device:C
- removed J? (x2): Screw_Terminal_01x02, symbol Connector:Screw_Terminal_01x02
- removed R? (x2): 1k, Resistor_SMD:R_0603_1608Metric, symbol Device:R
- removed R? (x2): 100, Resistor_SMD:R_0603_1608Metric, symbol Device:R
- removed U? (x2): FS8205A, Package_SO:TSSOP-8_4.4x3mm_P0.65mm, symbol Library:FS8205A
- removed U? (x2): DW01-P, Package_TO_SOT_SMD:SOT-23-6, symbol Library:DW01-P
- added C? (x2): 100n, Capacitor_SMD:C_0603_1608Metric, symbol Device:C
- added D? (x3): LED_ALT, LED_SMD:LED_0805_2012Metric, symbol Device:LED_ALT
- added J? (x2): Screw_Terminal_01x02, symbol Connector:Screw_Terminal_01x02
- added Q? (x3): Q_PMOS_GSD, Package_TO_SOT_SMD:SOT-23, symbol Device:Q_PMOS_GSD
- added R? (x5): 1k, Resistor_SMD:R_0603_1608Metric, symbol Device:R
- added R? (x3): 10k, Resistor_SMD:R_0603_1608Metric, symbol Device:R
- added R? (x2): 100, Resistor_SMD:R_0603_1608Metric, symbol Device:R
- added U? (x2): FS8205A, Package_SO:TSSOP-8_4.4x3mm_P0.65mm, symbol Library:FS8205A
- added U? (x2): DW01-P, Package_TO_SOT_SMD:SOT-23-6, symbol Library:DW01-P
Connections:
- wire segments 75 -> 104
Other:
- note removed: "Złącze na baterie"
- moved on the sheet: C?, D?, F?, J?, R?, SW?, U?

Commit message: Minor designator change.
Parts:
- removed D? (x3): LED_ALT, LED_SMD:LED_0805_2012Metric, symbol Device:LED_ALT
- added D? (x2): RED, LED_SMD:LED_0805_2012Metric, symbol Device:LED_ALT
- added D?: GREEN, LED_SMD:LED_0805_2012Metric, symbol Device:LED_ALT
- D?: value LED_ALT -> RED
Changed lines of the file:
@@
 Wire Wire Line
 	7450 2350 7800 2350
-$Comp
-L Device:LED_ALT D?
-U 1 1 5C638B5A
-P 5150 3200
-F 0 "D?" V 5142 3082 50  0000 R CNN
-F 1 "LED_ALT" V 5097 3082 50  0001 R CNN
-F 2 "LED_SMD:LED_0805_2012Metric" H 5150 3200 50  0001 C CNN
-F 3 "~" H 5150 3200 50  0001 C CNN
-	1    5150 3200
-	0    -1   -1   0
-$EndComp
 Wire Wire Line
 	4200 1350 4200 1400
@@
 U 1 1 5C6389A0
 P 2450 1650
-F 0 "D?" V 2442 1532 50  0000 R CNN
-F 1 "LED_ALT" V 2397 1532 50  0001 R CNN
+F 0 "D?" V 2450 1550 50  0000 R CNN
+F 1 "RED" V 2550 1600 50  0000 R CNN
 F 2 "LED_SMD:LED_0805_2012Metric" H 2450 1650 50  0001 C CNN
 F 3 "~" H 2450 1650 50  0001 C CNN
@@
 	-1   0    0    -1
 $EndComp
-$Comp
-L Device:LED_ALT D?
-U 1 1 5C68BD1E
-P 2450 3250
-F 0 "D?" V 2442 3132 50  0000 R CNN
-F 1 "LED_ALT" V 2397 3132 50  0001 R CNN
-F 2 "LED_SMD:LED_0805_2012Metric" H 2450 3250 50  0001 C CNN
-F 3 "~" H 2450 3250 50  0001 C CNN
-	1    2450 3250
-	0    1    1    0
-$EndComp
 Wire Wire Line
 	2200 3350 2200 3000
@@
 	1    2450 5150
 	-1   0    0    -1
-$EndComp
-$Comp
-L Device:LED_ALT D?
-U 1 1 5C693DFF
-P 2450 4850
-F 0 "D?" V 2442 4732 50  0000 R CNN
-F 1 "LED_ALT" V 2397 4732 50  0001 R CNN
-F 2 "LED_SMD:LED_0805_2012Metric" H 2450 4850 50  0001 C CNN
-F 3 "~" H 2450 4850 50  0001 C CNN
-	1    2450 4850
-	0    1    1    0
 $EndComp
 Wire Wire Line
@@
 	0    -1   -1   0
 $EndComp
+$Comp
+L Device:LED_ALT D?
+U 1 1 5C6C278F
+P 2450 3250
+F 0 "D?" V 2450 3150 50  0000 R CNN
+F 1 "RED" V 2550 3200 50  0000 R CNN
+F 2 "LED_SMD:LED_0805_2012Metric" H 2450 3250 50  0001 C CNN
+F 3 "~" H 2450 3250 50  0001 C CNN
+	1    2450 3250
+	0    1    1    0
+$EndComp
+$Comp
+L Device:LED_ALT D?
+U 1 1 5C6C2A59
+P 2450 4850
+F 0 "D?" V 2450 4750 50  0000 R CNN
+F 1 "RED" V 2550 4800 50  0000 R CNN
+F 2 "LED_SMD:LED_0805_2012Metric" H 2450 4850 50  0001 C CNN
+F 3 "~" H 2450 4850 50  0001 C CNN
+	1    2450 4850
+	0    1    1    0
+$EndComp
+$Comp
+L Device:LED_ALT D?
+U 1 1 5C6C368A
+P 5150 3200
+F 0 "D?" V 5200 3100 50  0000 R CNN
+F 1 "GREEN" V 5100 3100 50  0000 R CNN
+F 2 "LED_SMD:LED_0805_2012Metric" H 5150 3200 50  0001 C CNN
+F 3 "~" H 5150 3200 50  0001 C CNN
+	1    5150 3200
+	0    -1   -1   0
+$EndComp

Commit message: Removed varistors and added Atmega8 crystal resonator.
Squashed commit of the following:

commit fdff6d01c76f16de22ef88d4f0a11d1713a9c16b
Author: Paweł <mackipawel@gmail.com>
Date:   Sat Feb 23 19:48:33 2019 +0100

    Removed varistors and added Atmega8 crystal resonator.
Parts:
- removed RV? (x2): 18V, symbol Device:Varistor
Connections:
- wire segments 104 -> 100
Other:
- moved on the sheet: D?, J?
Changed lines of the file:
@@
 L Connector:Screw_Terminal_01x02 J?
 U 1 1 5C6116CB
-P 10000 1550
-F 0 "J?" H 9950 1650 50  0000 C CNN
-F 1 "Screw_Terminal_01x02" H 9920 1676 50  0001 C CNN
-F 2 "" H 10000 1550 50  0001 C CNN
-F 3 "~" H 10000 1550 50  0001 C CNN
-	1    10000 1550
+P 9700 1550
+F 0 "J?" H 9650 1650 50  0000 C CNN
+F 1 "Screw_Terminal_01x02" H 9620 1676 50  0001 C CNN
+F 2 "" H 9700 1550 50  0001 C CNN
+F 3 "~" H 9700 1550 50  0001 C CNN
+	1    9700 1550
 	1    0    0    -1
 $EndComp
@@
 L power:GND #PWR0104
 U 1 1 5C61B126
-P 9800 1850
-F 0 "#PWR0104" H 9800 1600 50  0001 C CNN
-F 1 "GND" H 9805 1677 50  0000 C CNN
-F 2 "" H 9800 1850 50  0001 C CNN
-F 3 "" H 9800 1850 50  0001 C CNN
-	1    9800 1850
+P 9500 1850
+F 0 "#PWR0104" H 9500 1600 50  0001 C CNN
+F 1 "GND" H 9505 1677 50  0000 C CNN
+F 2 "" H 9500 1850 50  0001 C CNN
+F 3 "" H 9500 1850 50  0001 C CNN
+	1    9500 1850
 	1    0    0    -1
 $EndComp
@@
 Connection ~ 5150 1850
 $Comp
-L Device:Varistor RV?
-U 1 1 5C66947E
+L Device:D_TVS_ALT D?
+U 1 1 5C6695A1
 P 6050 1700
-F 0 "RV?" H 6153 1746 50  0000 L CNN
-F 1 "18V" H 6153 1655 50  0000 L CNN
-F 2 "" V 5980 1700 50  0001 C CNN
+F 0 "D?" V 6050 1779 50  0000 L CNN
+F 1 "D_TVS_ALT" V 6095 1779 50  0001 L CNN
+F 2 "" H 6050 1700 50  0001 C CNN
 F 3 "~" H 6050 1700 50  0001 C CNN
 	1    6050 1700
-	1    0    0    -1
-$EndComp
-$Comp
-L Device:D_TVS_ALT D?
-U 1 1 5C6695A1
-P 6350 1700
-F 0 "D?" V 6350 1779 50  0000 L CNN
-F 1 "D_TVS_ALT" V 6395 1779 50  0001 L CNN
-F 2 "" H 6350 1700 50  0001 C CNN
-F 3 "~" H 6350 1700 50  0001 C CNN
-	1    6350 1700
 	0    1    1    0
 $EndComp
-Wire Wire Line
-	5600 1850 6050 1850
 Connection ~ 5600 1850
-Connection ~ 6050 1850
-Wire Wire Line
-	6050 1850 6350 1850
-Wire Wire Line
-	5600 1550 6050 1550
 Connection ~ 5600 1550
-Connection ~ 6050 1550
-Wire Wire Line
-	6050 1550 6350 1550
 $Comp
 L Device:C C?
@@
 $EndComp
 $Comp
-L Device:Varistor RV?
-U 1 1 5C66ED1E
+L Device:D_TVS_ALT D?
+U 1 1 5C66ED25
 P 8950 1700
-F 0 "RV?" H 9053 1746 50  0000 L CNN
-F 1 "18V" H 9053 1655 50  0000 L CNN
-F 2 "" V 8880 1700 50  0001 C CNN
+F 0 "D?" V 8950 1779 50  0000 L CNN
+F 1 "D_TVS_ALT" V 8995 1779 50  0001 L CNN
+F 2 "" H 8950 1700 50  0001 C CNN
 F 3 "~" H 8950 1700 50  0001 C CNN
 	1    8950 1700
-	1    0    0    -1
-$EndComp
-$Comp
-L Device:D_TVS_ALT D?
-U 1 1 5C66ED25
-P 9250 1700
-F 0 "D?" V 9250 1779 50  0000 L CNN
-F 1 "D_TVS_ALT" V 9295 1779 50  0001 L CNN
-F 2 "" H 9250 1700 50  0001 C CNN
-F 3 "~" H 9250 1700 50  0001 C CNN
-	1    9250 1700
 	0    1    1    0
 $EndComp
-Wire Wire Line
-	8500 1850 8950 1850
+Connection ~ 8500 1550
+Wire Wire Line
+	8250 1550 8500 1550
+Wire Wire Line
+	9500 1850 9500 1650
+Connection ~ 9500 1850
 Connection ~ 8950 1850
-Wire Wire Line
-	8950 1850 9250 1850
-Wire Wire Line
-	8500 1550 8950 1550
-Connection ~ 8500 1550
 Connection ~ 8950 1550
-Wire Wire Line
-	8950 1550 9250 1550
-Wire Wire Line
-	8250 1550 8500 1550
-Wire Wire Line
-	9800 1850 9800 1650
-Connection ~ 9800 1850
-Connection ~ 9250 1850
-Connection ~ 9250 1550
 Text Notes 5250 1250 0    50   ~ 0
 Zabezpieczenia napięcia baterii
@@
 L Device:D_ALT D?
 U 1 1 5C62AB5D
-P 9500 1700
-F 0 "D?" V 9500 1779 50  0000 L CNN
-F 1 "D_ALT" V 9545 1779 50  0001 L CNN
-F 2 "Diode_SMD:D_MiniMELF" H 9500 1700 50  0001 C CNN
-F 3 "~" H 9500 1700 50  0001 C CNN
-	1    9500 1700
+P 9200 1700
+F 0 "D?" V 9200 1779 50  0000 L CNN
+F 1 "D_ALT" V 9245 1779 50  0001 L CNN
+F 2 "Diode_SMD:D_MiniMELF" H 9200 1700 50  0001 C CNN
+F 3 "~" H 9200 1700 50  0001 C CNN
+	1    9200 1700
 	0    1    1    0
 $EndComp
 Wire Wire Line
-	9250 1550 9500 1550
-Wire Wire Line
-	9250 1850 9500 1850
+	8950 1550 9200 1550
+Wire Wire Line
+	8950 1850 9200 1850
 $Comp
 L Device:D_ALT D?
@@
 Wire Wire Line
 	8100 2350 8350 2350
-Connection ~ 9500 1550
-Wire Wire Line
-	9500 1550 9800 1550
-Connection ~ 9500 1850
-Wire Wire Line
-	9500 1850 9800 1850
+Connection ~ 9200 1550
+Wire Wire Line
+	9200 1550 9500 1550
+Connection ~ 9200 1850
+Wire Wire Line
+	9200 1850 9500 1850
 Wire Wire Line
 	7450 2350 7800 2350
@@
 	0    -1   -1   0
 $EndComp
+Wire Wire Line
+	5600 1550 6050 1550
+Wire Wire Line
+	5600 1850 6050 1850
+Wire Wire Line
+	8500 1550 8950 1550
+Wire Wire Line
+	8500 1850 8950 1850
 $EndSCHEMATC

Commit message: Footprint feature. Added some footprints to library.
Squashed commit of the following:

commit cd975fe41aefde478091de7f14ed38d0983c180d
Author: Paweł <mackipawel@gmail.com>
Date:   Tue Mar 26 21:11:20 2019 +0100

    Added RFM18 and 5MS1S102AM2QE footprints.

commit 4e602ef25fbcf5dd6c485f40bf8f72e3bcba2156
Merge: 6566fa8 80250b1
Author: Asiderr <norkam41@gmail.com>
Date:   Thu Mar 21 22:21:42 2019 +0100

    merge

commit 6566fa87254b74c1a8c88ea40d35451463bde8d8
Author: Asiderr <norkam41@gmail.com>
Date:   Thu Mar 21 22:13:41 2019 +0100

    Adding footprints of RJ9, DC/DC converter

commit 80250b18490f042be3a2014c95d5388371debc3d
Author: Paweł <mackipawel@gmail.com>
Date:   Thu Mar 21 22:08:10 2019 +0100

    Removed backup files from git.

commit 04658cd3c50c023263e023466e96f3f94a65df95
Merge: 7849973 bad73f3
Author: Paweł <mackipawel@gmail.com>
Date:   Thu Mar 21 22:07:23 2019 +0100

    Merge branch 'feature/footprints' of https://github.com/EcoTechTeam/Hardware into feature/footprints

commit 78499733d111ae0bedf73c4fca8fcef50fc29226
Author: Paweł <mackipawel@gmail.com>
Date:   Thu Mar 21 22:07:10 2019 +0100

    Fixed footprint library name to Footprints.

commit 3f8eab394080d79e7aead60b2eec59a08122afbc
Author: Paweł <mackipawel@gmail.com>
Date:   Thu Mar 21 21:19:44 2019 +0100

    Removed tables.

commit 684012423bea3414343087823362922cefb8473a
Merge: b428dfb 1892ec1
Author: Paweł <mackipawel@gmail.com>
Date:   Thu Mar 21 21:19:12 2019 +0100

    Merge

commit bad73f3c705cb3c30d3a26163545b978ffddeb4c
Author: Asiderr <norkam41@gmail.com>
Date:   Thu Mar 21 00:16:46 2019 +0100

    Adding footprints of pasives, diodes, transistors

commit 1892ec1f2bc7f41887eec779a92ff03034286e97
Author: Asiderr <norkam41@gmail.com>
Date:   Wed Mar 20 23:04:53 2019 +0100

    Adding footprints to System Supply

commit b428dfbf710c4231b032b3b85412e614af8e604a
Author: Paweł <mackipawel@gmail.com>
Date:   Wed Mar 20 22:59:15 2019 +0100

    Added few footprints.

commit c791dd8f20d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
Parts:
- removed J? (x3): Screw_Terminal_01x02, symbol Connector:Screw_Terminal_01x02
- removed K?: DIPxx-1Axx-11x, Relay_THT:Relay_StandexMeder_DIP_LowProfile, symbol Relay:DIPxx-1Axx-11x
- added J2, J4, J6, J7, J8, J9: Conn_01x01, Connector_Pin:Pin_D1.4mm_L8.5mm_W2.8mm_FlatFork, symbol Connector_Generic:Conn_01x01
- added K1: FRM18, symbol Library:FRM18
- C1: renamed from C?; value 100u -> 470u; footprint (none) -> Capacitor_THT:C_Radial_D10.0mm_H20.0mm_P5.00mm
- C3: renamed from C?; footprint (none) -> Capacitor_SMD:C_0805_2012Metric
- D2, D3: renamed from D?; footprint (none) -> Diode_SMD:D_SMC
- F1: renamed from F?; footprint (none) -> Footprints:Fuse_Blade
- J1, J3, J5: renamed from J?; footprint (none) -> Footprints:TerminalBlock_DG250_02P
- gave numbers to parts that had none: 29
Connections:
- wire segments 100 -> 94
