File: SafetySupply/SafetySupply.sch (KiCad schematic (older format))
At the start: 44 parts, among them J1 Screw_Terminal_01x02, J2 Conn_01x01, J3 Screw_Terminal_01x02, J4 Conn_01x01, J5 Screw_Terminal_01x02, J6 Conn_01x01, J7 Conn_01x01, J8 Conn_01x01, J9 Conn_01x01, K1 FRM18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

Commit message: Feature SafetySupply
Squashed commit of the following:

commit 9d5a0004d18ed8306ebf2eb05ad9a9ebf59c5dae
Author: Paweł <mackipawel@gmail.com>
Date:   Fri Mar 29 23:23:41 2019 +0100

    Small fixes
    .

commit b0d9d1a867e08e8066c55cc512f6fcb1bd2f5a2e
Author: Paweł <mackipawel@gmail.com>
Date:   Fri Mar 29 23:12:26 2019 +0100

    Added traces. Fixed some footprints.

commit b52da5269a39cad2ad8b91ecb01a5432155c2a6d
Author: Paweł <mackipawel@gmail.com>
Date:   Thu Mar 28 23:41:23 2019 +0100

    Added angled switch and fuse connector. Placed BMS elements in optimal positions.

commit afa6441a3853fc020fd761c7d7073267e37056dd
Author: Paweł <mackipawel@gmail.com>
Date:   Wed Mar 27 19:05:06 2019 +0100

    Initial element positioning.

commit d81fd4aefa0f9975d87eff3b6fb3fbd108abf68c
Author: Paweł <mackipawel@gmail.com>
Date:   Tue Mar 26 21:21:43 2019 +0100

    Fixed symbol librares and assigned footprints.
Parts:
- removed SW1: SW_SPST, symbol Switch:SW_SPST
- removed unit 2 of U1
- removed unit 3 of U1
- removed unit 2 of U2
- removed unit 3 of U2
- added SW1: SW_SPDT, Footprints:5MS1S102AM6QE, symbol Switch:SW_SPDT
- added U3, U5: DW01-P, Package_TO_SOT_SMD:SOT-23-6, symbol Library:DW01-P
- added U4, U6: FS8205A, Package_SO:TSSOP-8_4.4x3mm_P0.65mm, symbol Library:FS8205A
- F1: footprint Footprints:Fuse_Blade -> Footprints:Fuse_Blade_90
- K1: footprint (none) -> Footprints:RFM18
Connections:
- wire segments 94 -> 96
- no-connect marks 0 -> 3
Changed lines of the file:
@@
 	1    0    0    -1
 $EndComp
-Wire Wire Line
-	3150 2200 2950 2200
 $Comp
 L power:+12V #PWR0101
 U 1 1 5C5F7175
-P 4200 1350
-F 0 "#PWR0101" H 4200 1200 50  0001 C CNN
-F 1 "+12V" H 4215 1523 50  0000 C CNN
-F 2 "" H 4200 1350 50  0001 C CNN
-F 3 "" H 4200 1350 50  0001 C CNN
-	1    4200 1350
+P 4200 1300
+F 0 "#PWR0101" H 4200 1150 50  0001 C CNN
+F 1 "+12V" H 4215 1473 50  0000 C CNN
+F 2 "" H 4200 1300 50  0001 C CNN
+F 3 "" H 4200 1300 50  0001 C CNN
+	1    4200 1300
 	1    0    0    -1
 $EndComp
@@
 L power:GND #PWR0104
 U 1 1 5C61B126
-P 9500 1850
-F 0 "#PWR0104" H 9500 1600 50  0001 C CNN
-F 1 "GND" H 9505 1677 50  0000 C CNN
-F 2 "" H 9500 1850 50  0001 C CNN
-F 3 "" H 9500 1850 50  0001 C CNN
-	1    9500 1850
+P 8500 1850
+F 0 "#PWR0104" H 8500 1600 50  0001 C CNN
+F 1 "GND" H 8505 1677 50  0000 C CNN
+F 2 "" H 8500 1850 50  0001 C CNN
+F 3 "" H 8500 1850 50  0001 C CNN
+	1    8500 1850
 	1    0    0    -1
 $EndComp
@@
 $EndComp
 Wire Wire Line
-	2950 1900 3150 1900
-Wire Wire Line
 	4150 2500 4150 2600
 Wire Wire Line
@@
 Wire Wire Line
 	2950 2200 2950 2600
-$Comp
-L Switch:SW_SPST SW1
-U 1 1 5C650F11
-P 3800 1400
-F 0 "SW1" H 3800 1543 50  0000 C CNN
-F 1 "SW_SPST" H 3800 1544 50  0001 C CNN
-F 2 "" H 3800 1400 50  0001 C CNN
-F 3 "" H 3800 1400 50  0001 C CNN
-	1    3800 1400
-	1    0    0    -1
-$EndComp
-Wire Wire Line
-	4200 1400 4000 1400
+Wire Wire Line
+	4200 1300 4000 1300
 Text Notes 3600 1100 0    50   ~ 0
 Włącznik zasilania
@@
 F 0 "F1" V 3003 1400 50  0000 C CNN
 F 1 "Fuse" V 3094 1400 50  0000 C CNN
-F 2 "Footprints:Fuse_Blade" V 3130 1400 50  0001 C CNN
+F 2 "Footprints:Fuse_Blade_90" V 3130 1400 50  0001 C CNN
 F 3 "~" H 3200 1400 50  0001 C CNN
 	1    3200 1400
@@
 Wire Wire Line
 	9500 1850 9500 1650
-Connection ~ 9500 1850
 Connection ~ 8950 1850
 Connection ~ 8950 1550
@@
 Connection ~ 9200 1850
 Wire Wire Line
-	9200 1850 9500 1850
-Wire Wire Line
 	7450 2350 7800 2350
-Wire Wire Line
-	4200 1350 4200 1400
 $Comp
 L Device:R R2
@@
 Wire Wire Line
 	2950 1900 2950 1800
-Connection ~ 2950 1900
 Wire Wire Line
 	2950 1500 2950 1400
@@
 F 3 "~" H 4150 3950 50  0001 C CNN
 	1    4150 3950
-	1    0    0    -1
-$EndComp
-$Comp
-L Library:FS8205A U2
-U 2 1 5C68BCD7
-P 3600 4300
-F 0 "U2" H 3400 4150 50  0000 C CNN
-F 1 "FS8205A" H 3800 4150 50  0000 C CNN
-F 2 "Package_SO:TSSOP-8_4.4x3mm_P0.65mm" H 3400 4050 50  0001 C CNN
-F 3 "https://www.ic-fortune.com/upload/Download/FS8205A-DS-12_EN.pdf" H 3400 4050 50  0001 C CNN
-	2    3600 4300
 	1    0    0    -1
 $EndComp
@@
 	1    0    0    -1
 $EndComp
-Wire Wire Line
-	3150 3800 2950 3800
 Connection ~ 2950 3800
-$Comp
-L Library:DW01-P U1
-U 2 1 5C68BCF4
-P 3600 3650
-F 0 "U1" H 3300 3950 50  0000 C CNN
-F 1 "DW01-P" H 3900 3950 50  0000 C CNN
-F 2 "Package_TO_SOT_SMD:SOT-23-6" H 3350 3950 50  0001 C CNN
-F 3 "https://cdn.sparkfun.com/assets/learn_tutorials/2/5/1/DW01-P_DataSheet_V10.pdf" H 3350 3950 50  0001 C CNN
-	2    3600 3650
-	1    0    0    -1
-$EndComp
-Wire Wire Line
-	2950 3500 3150 3500
 Wire Wire Line
 	4150 4100 4150 4200
@@
 Wire Wire Line
 	2950 3500 2950 3400
-Connection ~ 2950 3500
 Wire Wire Line
 	2950 3100 2950 3000
@@
 F 3 "~" H 4150 5550 50  0001 C CNN
 	1    4150 5550
-	1    0    0    -1
-$EndComp
-$Comp
-L Library:FS8205A U2
-U 3 1 5C693DD1
-P 3600 5900
-F 0 "U2" H 3400 5750 50  0000 C CNN
-F 1 "FS8205A" H 3800 5750 50  0000 C CNN
-F 2 "Package_SO:TSSOP-8_4.4x3mm_P0.65mm" H 3400 5650 50  0001 C CNN
-F 3 "https://www.ic-fortune.com/upload/Download/FS8205A-DS-12_EN.pdf" H 3400 5650 50  0001 C CNN
-	3    3600 5900
 	1    0    0    -1
 $EndComp
@@
 	1    0    0    -1
 $EndComp
-Wire Wire Line
-	3150 5400 2950 5400
 Connection ~ 2950 5400
-$Comp
-L Library:DW01-P U1
-U 3 1 5C693DE8
-P 3600 5250
-F 0 "U1" H 3300 5550 50  0000 C CNN
-F 1 "DW01-P" H 3900 5550 50  0000 C CNN
-F 2 "Package_TO_SOT_SMD:SOT-23-6" H 3350 5550 50  0001 C CNN
-F 3 "https://cdn.sparkfun.com/assets/learn_tutorials/2/5/1/DW01-P_DataSheet_V10.pdf" H 3350 5550 50  0001 C CNN
-	3    3600 5250
-	1    0    0    -1
-$EndComp
-Wire Wire Line
-	2950 5100 3150 5100
 Wire Wire Line
 	4150 5700 4150 5800
@@
 Wire Wire Line
 	2950 5100 2950 5000
-Connection ~ 2950 5100
 Wire Wire Line
 	2950 4700 2950 4600
@@
 F 0 "K1" V 8417 1750 50  0000 C CNN
 F 1 "FRM18" V 8326 1750 50  0000 C CNN
-F 2 "" H 8300 1700 50  0001 L CNN
+F 2 "Footprints:RFM18" H 8300 1700 50  0001 L CNN
 F 3 "https://www.tme.eu/pl/Document/89b4103d1f3caa57a1b3e92993b9af62/FRM18.pdf?fbclid=IwAR2nivsTICXGdIlFtGx6DdiS3tLQJLmOYCGR6QBl4_J1FSsytW3mL1SHknk" H 7950 1750 50  0001 C CNN
 	1    7950 1750
 	0    1    -1   0
 $EndComp
+$Comp
+L Switch:SW_SPDT SW1
+U 1 1 5C9AB870
+P 3800 1400
+F 0 "SW1" H 3800 1593 50  0000 C CNN
+F 1 "SW_SPDT" H 3800 1594 50  0001 C CNN
+F 2 "Footprints:5MS1S102AM6QE" H 3800 1400 50  0001 C CNN
+F 3 "" H 3800 1400 50  0001 C CNN
+	1    3800 1400
+	1    0    0    1
+$EndComp
+$Comp
+L Library:DW01-P U3
+U 1 1 5C9B2C7B
+P 3600 3650
+F 0 "U3" H 3300 3950 50  0000 C CNN
+F 1 "DW01-P" H 3900 3950 50  0000 C CNN
+F 2 "Package_TO_SOT_SMD:SOT-23-6" H 3350 3950 50  0001 C CNN
+F 3 "https://cdn.sparkfun.com/assets/learn_tutorials/2/5/1/DW01-P_DataSheet_V10.pdf" H 3350 3950 50  0001 C CNN
+	1    3600 3650
+	1    0    0    -1
+$EndComp
+$Comp
+L Library:DW01-P U5
+U 1 1 5C9B5450
+P 3600 5250
+F 0 "U5" H 3300 5550 50  0000 C CNN
+F 1 "DW01-P" H 3900 5550 50  0000 C CNN
+F 2 "Package_TO_SOT_SMD:SOT-23-6" H 3350 5550 50  0001 C CNN
+F 3 "https://cdn.sparkfun.com/assets/learn_tutorials/2/5/1/DW01-P_DataSheet_V10.pdf" H 3350 5550 50  0001 C CNN
+	1    3600 5250
+	1    0    0    -1
+$EndComp
+$Comp
+L Library:FS8205A U4
+U 1 1 5C9B5500
+P 3600 4300
+F 0 "U4" H 3400 4150 50  0000 C CNN
+F 1 "FS8205A" H 3800 4150 50  0000 C CNN
+F 2 "Package_SO:TSSOP-8_4.4x3mm_P0.65mm" H 3400 4050 50  0001 C CNN
+F 3 "https://www.ic-fortune.com/upload/Download/FS8205A-DS-12_EN.pdf" H 3400 4050 50  0001 C CNN
+	1    3600 4300
+	1    0    0    -1
+$EndComp
+Connection ~ 3250 4200
+$Comp
+L Library:FS8205A U6
+U 1 1 5C9B55A6
+P 3600 5900
+F 0 "U6" H 3400 5750 50  0000 C CNN
+F 1 "FS8205A" H 3800 5750 50  0000 C CNN
+F 2 "Package_SO:TSSOP-8_4.4x3mm_P0.65mm" H 3400 5650 50  0001 C CNN
+F 3 "https://www.ic-fortune.com/upload/Download/FS8205A-DS-12_EN.pdf" H 3400 5650 50  0001 C CNN
+	1    3600 5900
+	1    0    0    -1
+$EndComp
+Connection ~ 3250 5800
+Wire Wire Line
+	2950 2200 3150 2200
+Wire Wire Line
+	2950 1900 3150 1900
+Connection ~ 2950 1900
+Wire Wire Line
+	2950 3800 3150 3800
+Wire Wire Line
+	2950 3500 3150 3500
+Connection ~ 2950 3500
+Wire Wire Line
+	2950 5100 3150 5100
+Connection ~ 2950 5100
+Wire Wire Line
+	2950 5400 3150 5400
+Wire Wire Line
+	9200 1850 9500 1850
+Connection ~ 8500 1850
+NoConn ~ 4150 3500
+NoConn ~ 4150 1900
+NoConn ~ 4150 5100
+Wire Wire Line
+	4000 1500 4000 1550
+Wire Wire Line
+	4000 1550 3600 1550
+Wire Wire Line
+	3600 1550 3600 1400
+Connection ~ 3600 1400
 $EndSCHEMATC

Commit message: Fixed silkscreen for SafetySupply, added mounting holes.
Parts:
- C1: footprint Capacitor_THT:C_Radial_D10.0mm_H20.0mm_P5.00mm -> Footprints:C_Radial_D10.0mm_H20.0mm_P5.00mm
Changed lines of the file:
@@
 EESchema Schematic File Version 4
-LIBS:SafetySupply-cache
 EELAYER 26 0
 EELAYER END
@@
 F 0 "C1" H 5268 1746 50  0000 L CNN
 F 1 "470u" H 5268 1655 50  0000 L CNN
-F 2 "Capacitor_THT:C_Radial_D10.0mm_H20.0mm_P5.00mm" H 5188 1550 50  0001 C CNN
+F 2 "Footprints:C_Radial_D10.0mm_H20.0mm_P5.00mm" H 5188 1550 50  0001 C CNN
 F 3 "~" H 5150 1700 50  0001 C CNN
 	1    5150 1700

Commit message: Removed Switches from bus devices and added mounting holes in schematics.
Squashed commit of the following:

commit 448b4f84a5f64686dc4334a0b6d81609891ca7cf
Author: Paweł <mackipawel@gmail.com>
Date:   Sun Apr 28 20:22:14 2019 +0200

    Added mouting holes to SystemSupply.

commit d45917b7024ecbe087cb8328a2c33d3ab10399ff
Author: Paweł <mackipawel@gmail.com>
Date:   Sun Apr 28 20:13:41 2019 +0200

    Added mouting holes to SafetySystem.

commit 6365380671305e2241dc821ec3b00ae08a997ac5
Author: Paweł <mackipawel@gmail.com>
Date:   Sun Apr 28 20:11:13 2019 +0200

    Added mouting holes to SafetySupply.

commit 00163d4bba61eb48f9ebb4c601b04017e78006be
Author: Paweł <mackipawel@gmail.com>
Date:   Sun Apr 28 20:06:38 2019 +0200

    Fixed MotorController.

commit ec0507ca51ef80aebbe2605505e7109beac59e98
Author: Paweł <mackipawel@gmail.com>
Date:   Sun Apr 28 19:54:40 2019 +0200

    Fixed MotorDriver.
Parts:
- added G1: EcoTechLogo, Footprints:EcoTech_small, symbol Library:EcoTechLogo
- added H1, H2: MountingHole, MountingHole:MountingHole_2.2mm_M2, symbol Mechanical:MountingHole
Changed lines of the file:
@@
 EESchema Schematic File Version 4
+LIBS:SafetySupply-cache
 EELAYER 26 0
 EELAYER END
@@
 	3600 1550 3600 1400
 Connection ~ 3600 1400
+$Comp
+L Library:EcoTechLogo G1
+U 1 1 5CC90702
+P 7100 5900
+F 0 "G1" H 7100 6000 50  0001 C CNN
+F 1 "EcoTechLogo" H 7125 5900 50  0000 L CNN
+F 2 "Footprints:EcoTech_small" H 7100 5900 50  0001 C CNN
+F 3 "" H 7100 5900 50  0001 C CNN
+	1    7100 5900
+	1    0    0    -1
+$EndComp
+$Comp
+L Mechanical:MountingHole H1
+U 1 1 5CC907BB
+P 7100 5550
+F 0 "H1" H 7200 5550 50  0000 L CNN
+F 1 "MountingHole" H 7200 5505 50  0001 L CNN
+F 2 "MountingHole:MountingHole_2.2mm_M2" H 7100 5550 50  0001 C CNN
+F 3 "~" H 7100 5550 50  0001 C CNN
+	1    7100 5550
+	1    0    0    -1
+$EndComp
+$Comp
+L Mechanical:MountingHole H2
+U 1 1 5CC90BEA
+P 7450 5550
+F 0 "H2" H 7550 5550 50  0000 L CNN
+F 1 "MountingHole" H 7550 5505 50  0001 L CNN
+F 2 "MountingHole:MountingHole_2.2mm_M2" H 7450 5550 50  0001 C CNN
+F 3 "~" H 7450 5550 50  0001 C CNN
+	1    7450 5550
+	1    0    0    -1
+$EndComp
 $EndSCHEMATC
