File: SafetySystem/SafetySystem.sch (KiCad schematic (older format))
At the start: 82 parts

Commit message: Removed varistors and added Atmega8 crystal resonator.
Squashed commit of the following:

commit fdff6d01c76f16de22ef88d4f0a11d1713a9c16b
Author: Paweł <mackipawel@gmail.com>
Date:   Sat Feb 23 19:48:33 2019 +0100

    Removed varistors and added Atmega8 crystal resonator.
Parts:
- removed RV?: 18V, symbol Device:Varistor
- added C? (x2): 100n, Capacitor_SMD:C_0603_1608Metric, symbol Device:C
- added Y?: 8Mhz, symbol Device:Crystal
Connections:
- wire segments 104 -> 105
Other:
- moved on the sheet: BZ?, C?, D?, J?, Q?, R?, SW?, U?

Commit message: Footprint feature. Added some footprints to library.
Squashed commit of the following:

commit cd975fe41aefde478091de7f14ed38d0983c180d
Author: Paweł <mackipawel@gmail.com>
Date:   Tue Mar 26 21:11:20 2019 +0100

    Added RFM18 and 5MS1S102AM2QE footprints.

commit 4e602ef25fbcf5dd6c485f40bf8f72e3bcba2156
Merge: 6566fa8 80250b1
Author: Asiderr <norkam41@gmail.com>
Date:   Thu Mar 21 22:21:42 2019 +0100

    merge

commit 6566fa87254b74c1a8c88ea40d35451463bde8d8
Author: Asiderr <norkam41@gmail.com>
Date:   Thu Mar 21 22:13:41 2019 +0100

    Adding footprints of RJ9, DC/DC converter

commit 80250b18490f042be3a2014c95d5388371debc3d
Author: Paweł <mackipawel@gmail.com>
Date:   Thu Mar 21 22:08:10 2019 +0100

    Removed backup files from git.

commit 04658cd3c50c023263e023466e96f3f94a65df95
Merge: 7849973 bad73f3
Author: Paweł <mackipawel@gmail.com>
Date:   Thu Mar 21 22:07:23 2019 +0100

    Merge branch 'feature/footprints' of https://github.com/EcoTechTeam/Hardware into feature/footprints

commit 78499733d111ae0bedf73c4fca8fcef50fc29226
Author: Paweł <mackipawel@gmail.com>
Date:   Thu Mar 21 22:07:10 2019 +0100

    Fixed footprint library name to Footprints.

commit 3f8eab394080d79e7aead60b2eec59a08122afbc
Author: Paweł <mackipawel@gmail.com>
Date:   Thu Mar 21 21:19:44 2019 +0100

    Removed tables.

commit 684012423bea3414343087823362922cefb8473a
Merge: b428dfb 1892ec1
Author: Paweł <mackipawel@gmail.com>
Date:   Thu Mar 21 21:19:12 2019 +0100

    Merge

commit bad73f3c705cb3c30d3a26163545b978ffddeb4c
Author: Asiderr <norkam41@gmail.com>
Date:   Thu Mar 21 00:16:46 2019 +0100

    Adding footprints of pasives, diodes, transistors

commit 1892ec1f2bc7f41887eec779a92ff03034286e97
Author: Asiderr <norkam41@gmail.com>
Date:   Wed Mar 20 23:04:53 2019 +0100

    Adding footprints to System Supply

commit b428dfbf710c4231b032b3b85412e614af8e604a
Author: Paweł <mackipawel@gmail.com>
Date:   Wed Mar 20 22:59:15 2019 +0100

    Added few footprints.

commit c791dd8f20d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
Parts:
- C? (x5): footprint (none) -> Capacitor_SMD:C_0603_1608Metric
- D?: footprint (none) -> Diode_SMD:D_SMC
- D? (x7): footprint (none) -> LED_SMD:LED_0805_2012Metric
- D? (x6): footprint (none) -> Diode_SMD:D_MiniMELF
- J? (x9): footprint (none) -> Footprints:TerminalBlock_DG250_02P
- L? (x2): footprint (none) -> Inductor_SMD:L_1812_4532Metric_Pad1.30x3.40mm_HandSolder
- Q? (x12): footprint (none) -> Package_TO_SOT_SMD:SOT-23
- R? (x25): footprint (none) -> Resistor_SMD:R_0603_1608Metric
- U?: symbol Library:MQ-8 -> SafetySystem-rescue:MQ-8-Library
- Y?: footprint (none) -> Crystal:Crystal_SMD_HC49-SD_HandSoldering

Commit message: Adding footprint of hydrogen sensor
Parts:
- SW?: footprint (none) -> Footprints:5MS1S102AM2QE
- U?: footprint (none) -> Footprints:MQ8_hydrogen_sens; symbol SafetySystem-rescue:MQ-8-Library -> SafetySystem-rescue:MQ-8-Library-SafetySystem-rescue
Changed lines of the file:
@@
 F 0 "SW?" H 1600 1243 50  0000 C CNN
 F 1 "SW_SPST" H 1600 1244 50  0001 C CNN
-F 2 "" H 1600 1100 50  0001 C CNN
+F 2 "Footprints:5MS1S102AM2QE" H 1600 1100 50  0001 C CNN
 F 3 "" H 1600 1100 50  0001 C CNN
 	1    1600 1100
@@
 $EndComp
 $Comp
-L SafetySystem-rescue:MQ-8-Library U?
+L SafetySystem-rescue:MQ-8-Library-SafetySystem-rescue U?
 U 1 1 5C6BF30D
 P 10000 2250
 F 0 "U?" H 9800 2450 50  0000 L CNN
 F 1 "MQ-8" H 10100 2100 50  0000 L CNN
-F 2 "" H 10000 2250 50  0001 C CNN
+F 2 "Footprints:MQ8_hydrogen_sens" H 10000 2250 50  0001 C CNN
 F 3 "https://dlnmh9ip6v2uc.cloudfront.net/datasheets/Sensors/Biometric/MQ-8.pdf" H 10000 2250 50  0001 C CNN
 	1    10000 2250

Commit message: Feature SafetySystem footprints.
Parts:
- removed SW?: SW_SPST, Footprints:5MS1S102AM2QE, symbol Switch:SW_SPST
- removed U?: LTV-817S, Package_DIP:SMDIP-4_W9.53mm, symbol Isolator:LTV-817S
- added SW?: SW_SPDT, Footprints:5MS1S102AM6QE, symbol Switch:SW_SPDT
- added U?: LTV-817S, Package_DIP:DIP-4_W7.62mm_LongPads, symbol Isolator:LTV-817S
- BZ?: footprint (none) -> Buzzer_Beeper:Buzzer_12x9.5RM7.6
- C? (x2): footprint Capacitor_SMD:C_0603_1608Metric -> Capacitor_SMD:C_0805_2012Metric
- C? (x2): value 100n -> 12p
- L?: value 4u7 -> 3u3; footprint Inductor_SMD:L_1812_4532Metric_Pad1.30x3.40mm_HandSolder -> Footprints:L_HPI0530-3R3
- SW?: footprint (none) -> Button_Switch_SMD:SW_SPST_TL3342
- SW? (x2): footprint (none) -> Button_Switch_THT:SW_PUSH-12mm
- U?: symbol SafetySystem-rescue:MQ-8-Library-SafetySystem-rescue -> Library:MQ-8
- U?: footprint Package_DIP:SMDIP-4_W9.53mm -> Package_DIP:DIP-4_W7.62mm_LongPads
- Y?: footprint Crystal:Crystal_SMD_HC49-SD_HandSoldering -> Crystal:Crystal_SMD_HC49-SD
Connections:
- wire segments 105 -> 108
Other:
- moved on the sheet: J?
Changed lines of the file:
@@
 EESchema Schematic File Version 4
-LIBS:SafetySystem-cache
 EELAYER 26 0
 EELAYER END
@@
 L Connector:Screw_Terminal_01x02 J?
 U 1 1 5C69DAF9
-P 1200 1100
-F 0 "J?" H 1120 1225 50  0000 C CNN
-F 1 "Screw_Terminal_01x02" H 1120 1226 50  0001 C CNN
-F 2 "Footprints:TerminalBlock_DG250_02P" H 1200 1100 50  0001 C CNN
-F 3 "~" H 1200 1100 50  0001 C CNN
-	1    1200 1100
+P 1200 1200
+F 0 "J?" H 1120 1325 50  0000 C CNN
+F 1 "Screw_Terminal_01x02" H 1120 1326 50  0001 C CNN
+F 2 "Footprints:TerminalBlock_DG250_02P" H 1200 1200 50  0001 C CNN
+F 3 "~" H 1200 1200 50  0001 C CNN
+	1    1200 1200
 	-1   0    0    -1
 $EndComp
@@
 	1    0    0    -1
 $EndComp
-Wire Wire Line
-	1400 1200 1400 1700
 $Comp
 L Device:Q_PMOS_GSD Q?
@@
 F 0 "C?" H 3815 1396 50  0000 L CNN
 F 1 "10u" H 3815 1305 50  0000 L CNN
-F 2 "Capacitor_SMD:C_0603_1608Metric" H 3738 1200 50  0001 C CNN
+F 2 "Capacitor_SMD:C_0805_2012Metric" H 3738 1200 50  0001 C CNN
 F 3 "~" H 3700 1350 50  0001 C CNN
 	1    3700 1350
@@
 P 5650 1100
 F 0 "L?" V 5875 1100 50  0000 C CNN
-F 1 "4u7" V 5784 1100 50  0000 C CNN
-F 2 "Inductor_SMD:L_1812_4532Metric_Pad1.30x3.40mm_HandSolder" H 5650 1100 50  0001 C CNN
-F 3 "~" H 5650 1100 50  0001 C CNN
+F 1 "3u3" V 5784 1100 50  0000 C CNN
+F 2 "Footprints:L_HPI0530-3R3" H 5650 1100 50  0001 C CNN
+F 3 "https://www.tme.eu/pl/details/hpi0530-3r3/dlawiki-smd-mocy/ferrocore/" H 5650 1100 50  0001 C CNN
 	1    5650 1100
 	0    -1   -1   0
@@
 F 0 "C?" H 6165 1496 50  0000 L CNN
 F 1 "10u" H 6165 1405 50  0000 L CNN
-F 2 "Capacitor_SMD:C_0603_1608Metric" H 6088 1300 50  0001 C CNN
+F 2 "Capacitor_SMD:C_0805_2012Metric" H 6088 1300 50  0001 C CNN
 F 3 "~" H 6050 1450 50  0001 C CNN
 	1    6050 1450
@@
 $EndComp
 Connection ~ 3700 1100
-$Comp
-L Switch:SW_SPST SW?
-U 1 1 5C6A54E1
-P 1600 1100
-F 0 "SW?" H 1600 1243 50  0000 C CNN
-F 1 "SW_SPST" H 1600 1244 50  0001 C CNN
-F 2 "Footprints:5MS1S102AM2QE" H 1600 1100 50  0001 C CNN
-F 3 "" H 1600 1100 50  0001 C CNN
-	1    1600 1100
-	1    0    0    -1
-$EndComp
 Wire Wire Line
 	1400 1700 2000 1700
@@
 F 0 "SW?" H 7850 1643 50  0000 C CNN
 F 1 "SW_Push" H 7850 1644 50  0001 C CNN
-F 2 "" H 7850 1650 50  0001 C CNN
+F 2 "Button_Switch_SMD:SW_SPST_TL3342" H 7850 1650 50  0001 C CNN
 F 3 "" H 7850 1650 50  0001 C CNN
 	1    7850 1450
@@
 $EndComp
 $Comp
-L SafetySystem-rescue:MQ-8-Library-SafetySystem-rescue U?
+L Library:MQ-8 U?
 U 1 1 5C6BF30D
 P 10000 2250
@@
 F 0 "BZ?" H 9353 5529 50  0000 L CNN
 F 1 "Buzzer" H 9353 5438 50  0000 L CNN
-F 2 "" V 9175 5600 50  0001 C CNN
+F 2 "Buzzer_Beeper:Buzzer_12x9.5RM7.6" V 9175 5600 50  0001 C CNN
 F 3 "~" V 9175 5600 50  0001 C CNN
 	1    9200 5500
@@
 F 0 "SW?" H 3450 3100 50  0000 C CNN
 F 1 "SW_Push" H 3450 3394 50  0001 C CNN
-F 2 "" H 3450 3400 50  0001 C CNN
+F 2 "Button_Switch_THT:SW_PUSH-12mm" H 3450 3400 50  0001 C CNN
 F 3 "" H 3450 3400 50  0001 C CNN
 	1    3450 3200
@@
 F 0 "U?" H 1650 6600 50  0000 C CNN
 F 1 "LTV-817S" H 1800 6634 50  0001 C CNN
-F 2 "Package_DIP:SMDIP-4_W9.53mm" H 1800 6100 50  0001 C CNN
-F 3 "http://www.us.liteon.com/downloads/LTV-817-827-847.PDF" H 1450 6700 50  0001 C CNN
+F 2 "Package_DIP:DIP-4_W7.62mm_LongPads" H 1800 6100 50  0001 C CNN
+F 3 "https://www.tme.eu/pl/details/fod817c/transoptory-wyjscie-cyfrowe/on-semiconductor-fairchild/" H 1450 6700 50  0001 C CNN
 	1    1800 6400
 	1    0    0    -1
@@
 F 0 "SW?" V 2700 6500 50  0000 C CNN
 F 1 "SW_Push" H 2700 6794 50  0001 C CNN
-F 2 "" H 2700 6800 50  0001 C CNN
+F 2 "Button_Switch_THT:SW_PUSH-12mm" H 2700 6800 50  0001 C CNN
 F 3 "" H 2700 6800 50  0001 C CNN
 	1    2700 6600
@@
 $EndComp
 $Comp
-L Isolator:LTV-817S U?
-U 1 1 5C80275A
-P 5100 6400
-F 0 "U?" H 5100 6725 50  0000 C CNN
-F 1 "LTV-817S" H 5100 6634 50  0000 C CNN
-F 2 "Package_DIP:SMDIP-4_W9.53mm" H 5100 6100 50  0001 C CNN
-F 3 "http://www.us.liteon.com/downloads/LTV-817-827-847.PDF" H 4750 6700 50  0001 C CNN
-	1    5100 6400
-	1    0    0    -1
-$EndComp
-$Comp
 L Device:Q_NMOS_GSD Q?
 U 1 1 5C802761
@@
 	1    0    0    -1
 $EndComp
-Connection ~ 5400 6500
 Wire Wire Line
 	5400 6200 5400 6300
@@
 F 0 "Y?" H 7300 1900 50  0000 C CNN
 F 1 "8Mhz" H 7250 1800 50  0000 C CNN
-F 2 "Crystal:Crystal_SMD_HC49-SD_HandSoldering" H 7550 1850 50  0001 C CNN
+F 2 "Crystal:Crystal_SMD_HC49-SD" H 7550 1850 50  0001 C CNN
 F 3 "~" H 7550 1850 50  0001 C CNN
 	1    7550 1850
@@
 P 7400 2050
 F 0 "C?" H 7515 2096 50  0000 L CNN
-F 1 "100n" H 7515 2005 50  0000 L CNN
+F 1 "12p" H 7515 2005 50  0000 L CNN
 F 2 "Capacitor_SMD:C_0603_1608Metric" H 7438 1900 50  0001 C CNN
 F 3 "~" H 7400 2050 50  0001 C CNN
@@
 P 7700 2050
 F 0 "C?" H 7750 2150 50  0000 L CNN
-F 1 "100n" H 7750 1900 50  0000 L CNN
+F 1 "12p" H 7800 2000 50  0000 L CNN
 F 2 "Capacitor_SMD:C_0603_1608Metric" H 7738 1900 50  0001 C CNN
 F 3 "~" H 7700 2050 50  0001 C CNN
@@
 Wire Wire Line
 	2200 1100 2350 1100
+$Comp
+L Switch:SW_SPDT SW?
+U 1 1 5C9FE7C5
+P 1600 1200
+F 0 "SW?" H 1600 1393 50  0000 C CNN
+F 1 "SW_SPDT" H 1600 1394 50  0001 C CNN
+F 2 "Footprints:5MS1S102AM6QE" H 1600 1200 50  0001 C CNN
+F 3 "" H 1600 1200 50  0001 C CNN
+	1    1600 1200
+	1    0    0    -1
+$EndComp
+Wire Wire Line
+	1800 1300 1800 1400
+Wire Wire Line
+	1400 1300 1400 1400
+Wire Wire Line
+	1400 1400 1800 1400
+Connection ~ 1400 1400
+Wire Wire Line
+	1400 1400 1400 1700
+$Comp
+L Isolator:LTV-817S U?
+U 1 1 5CA27408
+P 5100 6400
+F 0 "U?" H 4950 6600 50  0000 C CNN
+F 1 "LTV-817S" H 5100 6634 50  0001 C CNN
+F 2 "Package_DIP:DIP-4_W7.62mm_LongPads" H 5100 6100 50  0001 C CNN
+F 3 "https://www.tme.eu/pl/details/fod817c/transoptory-wyjscie-cyfrowe/on-semiconductor-fairchild/" H 4750 6700 50  0001 C CNN
+	1    5100 6400
+	1    0    0    -1
+$EndComp
+Connection ~ 5400 6500
 $EndSCHEMATC

Commit message: Feature schematic annotation
Squashed commit of the following:

commit aec2ebb03e2dc3915f631c1ed1dd696ff1568698
Author: Paweł <mackipawel@gmail.com>
Date:   Sat Mar 30 14:48:59 2019 +0100

    Annotated schematic.
Parts:
- NT1: renamed from NT?; footprint (none) -> NetTie:NetTie-2_SMD_Pad0.5mm
- gave numbers to parts that had none: 83
Connections:
- no-connect marks 0 -> 15

Commit message: Finished SafetySystem PCB.
Parts:
- removed SW1: SW_SPDT, Footprints:5MS1S102AM6QE, symbol Switch:SW_SPDT
- added C9: 100n, Capacitor_SMD:C_0603_1608Metric, symbol Device:C
- C1: footprint Capacitor_SMD:C_0805_2012Metric -> Capacitor_SMD:C_1206_3216Metric
- C2: value 100n -> 4u7; footprint Capacitor_SMD:C_0603_1608Metric -> Capacitor_SMD:C_0805_2012Metric
- C3: value 10u -> 22u; footprint Capacitor_SMD:C_0805_2012Metric -> Capacitor_SMD:C_1210_3225Metric
- J4: footprint Connector_IDC:IDC-Header_2x05_P2.54mm_Horizontal -> Connector_IDC:IDC-Header_2x05_P2.54mm_Vertical
- L2: footprint Inductor_SMD:L_1812_4532Metric_Pad1.30x3.40mm_HandSolder -> Inductor_SMD:L_0805_2012Metric_Pad1.15x1.40mm_HandSolder
Connections:
- wire segments 108 -> 109
Other:
- moved on the sheet: D1, J1
Changed lines of the file:
@@
 L Connector:Screw_Terminal_01x02 J1
 U 1 1 5C69DAF9
-P 1200 1200
-F 0 "J1" H 1120 1325 50  0000 C CNN
-F 1 "Screw_Terminal_01x02" H 1120 1326 50  0001 C CNN
-F 2 "Footprints:TerminalBlock_DG250_02P" H 1200 1200 50  0001 C CNN
-F 3 "~" H 1200 1200 50  0001 C CNN
-	1    1200 1200
+P 1150 1200
+F 0 "J1" H 1070 1325 50  0000 C CNN
+F 1 "Screw_Terminal_01x02" H 1070 1326 50  0001 C CNN
+F 2 "Footprints:TerminalBlock_DG250_02P" H 1150 1200 50  0001 C CNN
+F 3 "~" H 1150 1200 50  0001 C CNN
+	1    1150 1200
 	-1   0    0    -1
 $EndComp
@@
 L Device:D_TVS_ALT D1
 U 1 1 5C69E385
-P 2350 1400
-F 0 "D1" V 2350 1479 50  0000 L CNN
-F 1 "D_TVS_ALT" V 2395 1479 50  0001 L CNN
-F 2 "Diode_SMD:D_SMC" H 2350 1400 50  0001 C CNN
-F 3 "~" H 2350 1400 50  0001 C CNN
-	1    2350 1400
+P 1700 1400
+F 0 "D1" V 1700 1479 50  0000 L CNN
+F 1 "D_TVS_ALT" V 1745 1479 50  0001 L CNN
+F 2 "Diode_SMD:D_SMC" H 1700 1400 50  0001 C CNN
+F 3 "~" H 1700 1400 50  0001 C CNN
+	1    1700 1400
 	0    1    1    0
 $EndComp
 Wire Wire Line
-	2350 1100 2350 1250
-Wire Wire Line
-	2350 1550 2350 1700
+	1700 1100 1700 1250
+Wire Wire Line
+	1700 1550 1700 1700
 $Comp
 L power:+12V #PWR0102
@@
 	1    0    0    -1
 $EndComp
-Connection ~ 2350 1100
 Text Notes 2200 1900 0    50   ~ 0
 Zabezpieczenie zasilania
@@
 P 4050 1350
 F 0 "C2" H 4165 1396 50  0000 L CNN
-F 1 "100n" H 4165 1305 50  0000 L CNN
-F 2 "Capacitor_SMD:C_0603_1608Metric" H 4088 1200 50  0001 C CNN
+F 1 "4u7" H 4165 1305 50  0000 L CNN
+F 2 "Capacitor_SMD:C_0805_2012Metric" H 4088 1200 50  0001 C CNN
 F 3 "~" H 4050 1350 50  0001 C CNN
 	1    4050 1350
@@
 F 0 "C1" H 3815 1396 50  0000 L CNN
 F 1 "10u" H 3815 1305 50  0000 L CNN
-F 2 "Capacitor_SMD:C_0805_2012Metric" H 3738 1200 50  0001 C CNN
+F 2 "Capacitor_SMD:C_1206_3216Metric" H 3738 1200 50  0001 C CNN
 F 3 "~" H 3700 1350 50  0001 C CNN
 	1    3700 1350
@@
 P 6050 1450
 F 0 "C3" H 6165 1496 50  0000 L CNN
-F 1 "10u" H 6165 1405 50  0000 L CNN
-F 2 "Capacitor_SMD:C_0805_2012Metric" H 6088 1300 50  0001 C CNN
+F 1 "22u" H 6165 1405 50  0000 L CNN
+F 2 "Capacitor_SMD:C_1210_3225Metric" H 6088 1300 50  0001 C CNN
 F 3 "~" H 6050 1450 50  0001 C CNN
 	1    6050 1450
@@
 $EndComp
 Connection ~ 3700 1100
-Wire Wire Line
-	1400 1700 2000 1700
 Text Notes 1400 850  0    50   ~ 0
 Włącznik\nzasilania
@@
 	0    -1   -1   0
 $EndComp
-Wire Wire Line
-	2600 1100 2350 1100
 Connection ~ 2600 1100
-Wire Wire Line
-	2600 1700 2350 1700
-Connection ~ 2350 1700
 $Comp
 L power:GND #PWR0111
@@
 F 0 "L2" V 6290 2350 50  0000 C CNN
 F 1 "10u" V 6199 2350 50  0000 C CNN
-F 2 "Inductor_SMD:L_1812_4532Metric_Pad1.30x3.40mm_HandSolder" H 6100 2350 50  0001 C CNN
+F 2 "Inductor_SMD:L_0805_2012Metric_Pad1.15x1.40mm_HandSolder" H 6100 2350 50  0001 C CNN
 F 3 "~" H 6100 2350 50  0001 C CNN
 	1    6100 2350
@@
 	1    0    0    -1
 $EndComp
-$Comp
-L power:GND #PWR0112
-U 1 1 5C6A1CBD
-P 5850 2650
-F 0 "#PWR0112" H 5850 2400 50  0001 C CNN
-F 1 "GND" H 5855 2477 50  0000 C CNN
-F 2 "" H 5850 2650 50  0001 C CNN
-F 3 "" H 5850 2650 50  0001 C CNN
-	1    5850 2650
-	1    0    0    -1
-$EndComp
 Wire Wire Line
 	5850 2350 5950 2350
@@
 L power:+5V #PWR0113
 U 1 1 5C6A25E9
-P 5850 2350
-F 0 "#PWR0113" H 5850 2200 50  0001 C CNN
-F 1 "+5V" H 5865 2523 50  0000 C CNN
-F 2 "" H 5850 2350 50  0001 C CNN
-F 3 "" H 5850 2350 50  0001 C CNN
-	1    5850 2350
+P 5600 2350
+F 0 "#PWR0113" H 5600 2200 50  0001 C CNN
+F 1 "+5V" H 5615 2523 50  0000 C CNN
+F 2 "" H 5600 2350 50  0001 C CNN
+F 3 "" H 5600 2350 50  0001 C CNN
+	1    5600 2350
 	1    0    0    -1
 $EndComp
@@
 Wire Wire Line
 	6000 2650 5850 2650
-Connection ~ 5850 2650
 Wire Wire Line
 	6200 2650 6350 2650
@@
 $EndComp
 $Comp
-L Library:MQ-8 U2
-U 1 1 5C6BF30D
-P 10000 2250
-F 0 "U2" H 9800 2450 50  0000 L CNN
-F 1 "MQ-8" H 10100 2100 50  0000 L CNN
-F 2 "Footprints:MQ8_hydrogen_sens" H 10000 2250 50  0001 C CNN
-F 3 "https://dlnmh9ip6v2uc.cloudfront.net/datasheets/Sensors/Biometric/MQ-8.pdf" H 10000 2250 50  0001 C CNN
-	1    10000 2250
-	1    0    0    -1
-$EndComp
-$Comp
-L power:+5V #PWR0128
-U 1 1 5C6C226F
-P 10000 2000
-F 0 "#PWR0128" H 10000 1850 50  0001 C CNN
-F 1 "+5V" H 10015 2173 50  0000 C CNN
-F 2 "" H 10000 2000 50  0001 C CNN
-F 3 "" H 10000 2000 50  0001 C CNN
-	1    10000 2000
-	1    0    0    -1
-$EndComp
-$Comp
-L power:GND #PWR0129
-U 1 1 5C6C2428
-P 10000 2550
-F 0 "#PWR0129" H 10000 2300 50  0001 C CNN
-F 1 "GND" H 10005 2377 50  0000 C CNN
-F 2 "" H 10000 2550 50  0001 C CNN
-F 3 "" H 10000 2550 50  0001 C CNN
-	1    10000 2550
-	1    0    0    -1
-$EndComp
-$Comp
 L Device:R R7
 U 1 1 5C6C2AFB
@@
 	-1   0    0    -1
 $EndComp
-$Comp
-L power:GND #PWR0130
-U 1 1 5C6C2BB1
-P 9750 2550
-F 0 "#PWR0130" H 9750 2300 50  0001 C CNN
-F 1 "GND" H 9755 2377 50  0000 C CNN
-F 2 "" H 9750 2550 50  0001 C CNN
-F 3 "" H 9750 2550 50  0001 C CNN
-	1    9750 2550
-	1    0    0    -1
-$EndComp
 Wire Wire Line
 	10000 2550 10000 2500
-Connection ~ 9750 2250
 Text Label 9700 2250 2    50   ~ 0
 ADC
@@
 F 0 "J4" H 10750 6100 50  0000 R CNN
 F 1 "AVR-ISP-10" H 10221 5705 50  0001 R CNN
-F 2 "Connector_IDC:IDC-Header_2x05_P2.54mm_Horizontal" V 10250 5750 50  0001 C CNN
+F 2 "Connector_IDC:IDC-Header_2x05_P2.54mm_Vertical" V 10250 5750 50  0001 C CNN
 F 3 " ~" H 9225 5150 50  0001 C CNN
 	1    10500 5700
 	-1   0    0    -1
 $EndComp
-Wire Wire Line
-	10250 2000 10000 2000
-Connection ~ 10000 2000
 Wire Wire Line
 	9500 2250 9750 2250
@@
 $EndComp
 $Comp
-L power:GNDA #PWR01
-U 1 1 5C72A1D7
-P 7400 2200
-F 0 "#PWR01" H 7400 1950 50  0001 C CNN
-F 1 "GNDA" H 7405 2027 50  0000 C CNN
-F 2 "" H 7400 2200 50  0001 C CNN
-F 3 "" H 7400 2200 50  0001 C CNN
-	1    7400 2200
-	1    0    0    -1
-$EndComp
-$Comp
 L Device:C C5
 U 1 1 5C72D4D1
@@
 	1    0    0    -1
 $EndComp
-$Comp
-L power:GNDA #PWR02
-U 1 1 5C72D4D8
-P 7700 2200
-F 0 "#PWR02" H 7700 1950 50  0001 C CNN
-F 1 "GNDA" H 7705 2027 50  0000 C CNN
-F 2 "" H 7700 2200 50  0001 C CNN
-F 3 "" H 7700 2200 50  0001 C CNN
-	1    7700 2200
-	1    0    0    -1
-$EndComp
 Wire Wire Line
 	7700 1850 7700 1900
@@
 	7400 1650 7400 1850
 Connection ~ 7400 1850
-Wire Wire Line
-	2000 1700 2350 1700
-Wire Wire Line
-	2200 1100 2350 1100
-$Comp
-L Switch:SW_SPDT SW1
-U 1 1 5C9FE7C5
-P 1600 1200
-F 0 "SW1" H 1600 1393 50  0000 C CNN
-F 1 "SW_SPDT" H 1600 1394 50  0001 C CNN
-F 2 "Footprints:5MS1S102AM6QE" H 1600 1200 50  0001 C CNN
-F 3 "" H 1600 1200 50  0001 C CNN
-	1    1600 1200
-	1    0    0    -1
-$EndComp
-Wire Wire Line
-	1800 1300 1800 1400
-Wire Wire Line
-	1400 1300 1400 1400
-Wire Wire Line
-	1400 1400 1800 1400
-Connection ~ 1400 1400
-Wire Wire Line
-	1400 1400 1400 1700
 $Comp
 L Isolator:LTV-817S U5
@@
 NoConn ~ 8300 2350
 NoConn ~ 4500 1300
+$Comp
+L Device:C C9
+U 1 1 5CA05F43
+P 5600 2500
+F 0 "C9" H 5715 2546 50  0000 L CNN
+F 1 "100n" H 5715 2455 50  0000 L CNN
+F 2 "Capacitor_SMD:C_0603_1608Metric" H 5638 2350 50  0001 C CNN
+F 3 "~" H 5600 2500 50  0001 C CNN
+	1    5600 2500
+	-1   0    0    -1
+$EndComp
+$Comp
+L power:GND #PWR023
+U 1 1 5CA05F4A
+P 5600 2650
+F 0 "#PWR023" H 5600 2400 50  0001 C CNN
+F 1 "GND" H 5605 2477 50  0000 C CNN
+F 2 "" H 5600 2650 50  0001 C CNN
+F 3 "" H 5600 2650 50  0001 C CNN
+	1    5600 2650
+	1    0    0    -1
+$EndComp
+Wire Wire Line
+	5600 2350 5850 2350
+Wire Wire Line
+	5850 2650 5600 2650
+Connection ~ 5850 2650
+Connection ~ 5600 2650
+Connection ~ 5600 2350
+$Comp
+L power:GNDA #PWR0112
+U 1 1 5CA1826A
+P 9750 2550
+F 0 "#PWR0112" H 9750 2300 50  0001 C CNN
+F 1 "GNDA" H 9850 2400 50  0000 C CNN
+F 2 "" H 9750 2550 50  0001 C CNN
+F 3 "" H 9750 2550 50  0001 C CNN
+	1    9750 2550
+	1    0    0    -1
+$EndComp
+$Comp
+L power:GND #PWR0128
+U 1 1 5CA1857E
+P 10000 2550
+F 0 "#PWR0128" H 10000 2300 50  0001 C CNN
+F 1 "GND" H 9900 2400 50  0000 C CNN
+F 2 "" H 10000 2550 50  0001 C CNN
+F 3 "" H 10000 2550 50  0001 C CNN
+	1    10000 2550
+	-1   0    0    -1
+$EndComp
+$Comp
+L power:+5VA #PWR0129
+U 1 1 5CA1C2B6
+P 10250 2000
+F 0 "#PWR0129" H 10250 1850 50  0001 C CNN
+F 1 "+5VA" H 10300 2150 50  0000 C CNN
+F 2 "" H 10250 2000 50  0001 C CNN
+F 3 "" H 10250 2000 50  0001 C CNN
+	1    10250 2000
+	1    0    0    -1
+$EndComp
+$Comp
+L power:+5V #PWR0130
+U 1 1 5CA1C4C9
+P 10000 2000
+F 0 "#PWR0130" H 10000 1850 50  0001 C CNN
+F 1 "+5V" H 9950 2150 50  0000 C CNN
+F 2 "" H 10000 2000 50  0001 C CNN
+F 3 "" H 10000 2000 50  0001 C CNN
+	1    10000 2000
+	1    0    0    -1
+$EndComp
+Wire Wire Line
+	1350 1300 1350 1700
+Wire Wire Line
+	1350 1700 1700 1700
+Wire Wire Line
+	1350 1200 1400 1200
+Connection ~ 1700 1700
+Wire Wire Line
+	1700 1700 2000 1700
+Wire Wire Line
+	2000 1700 2600 1700
+Wire Wire Line
+	2200 1100 2600 1100
+Wire Wire Line
+	1800 1100 1700 1100
+Wire Wire Line
+	1400 1100 1400 1200
+Connection ~ 1700 1100
+Wire Wire Line
+	1700 1100 1400 1100
+$Comp
+L power:GND #PWR0134
+U 1 1 5CC0D9E6
+P 7400 2200
+F 0 "#PWR0134" H 7400 1950 50  0001 C CNN
+F 1 "GND" H 7405 2027 50  0000 C CNN
+F 2 "" H 7400 2200 50  0001 C CNN
+F 3 "" H 7400 2200 50  0001 C CNN
+	1    7400 2200
+	1    0    0    -1
+$EndComp
+$Comp
+L power:GND #PWR0135
+U 1 1 5CC0DA99
+P 7700 2200
+F 0 "#PWR0135" H 7700 1950 50  0001 C CNN
+F 1 "GND" H 7705 2027 50  0000 C CNN
+F 2 "" H 7700 2200 50  0001 C CNN
+F 3 "" H 7700 2200 50  0001 C CNN
+	1    7700 2200
+	1    0    0    -1
+$EndComp
+$Comp
+L Library:MQ-8 U2
+U 1 1 5CC4E574
+P 10000 2250
+F 0 "U2" H 10291 2296 50  0000 L CNN
+F 1 "MQ-8" H 10291 2205 50  0000 L CNN
+F 2 "Footprints:MQ8_hydrogen_sens" H 10000 2250 50  0001 C CNN
+F 3 "https://dlnmh9ip6v2uc.cloudfront.net/datasheets/Sensors/Biometric/MQ-8.pdf" H 10000 2250 50  0001 C CNN
+	1    10000 2250
+	1    0    0    -1
+$EndComp
+Connection ~ 9750 2250
 $EndSCHEMATC
