File: SafetySystem/SafetySystem.sch (KiCad schematic (older format))
At the start: 84 parts, among them J1 Screw_Terminal_01x02, J10 Screw_Terminal_01x02, J2 Screw_Terminal_01x02, J3 Screw_Terminal_01x02, J4 AVR-ISP-10, J5 Screw_Terminal_01x02, J6 Screw_Terminal_01x02, J7 Screw_Terminal_01x02, J8 Screw_Terminal_01x02, J9 Screw_Terminal_01x02, Q1 Q_PMOS_GSD, Q10 Q_NMOS_GSD, Q11 Q_NMOS_GSD, Q12 Q_NMOS_GSD, Q2 Q_PMOS_GSD, Q3 Q_PMOS_GSD, Q4 Q_NMOS_GSD, Q5 Q_NMOS_GSD, Q6 Q_NMOS_GSD, Q7 Q_NMOS_GSD, Q8 Q_NMOS_GSD, Q9 Q_NMOS_GSD, SW2 SW_Push, SW3 SW_Push, SW4 SW_Push, U1 ST1S10PHR, U2 MQ-8, U3 ATmega8A-AU, U4 LTV-817S, U5 LTV-817S, Y1 8Mhz

Commit message: SafetySystem potentiometer.
Squashed commit of the following:

commit c85b31eae362b98e5e9037a9aad6a815148d0818
Author: Paweł <mackipawel@gmail.com>
Date:   Sun Apr 28 12:07:02 2019 +0200

    Added potentiometer to the SafetySysytem.
Parts:
- removed NT1: Net-Tie_2, NetTie:NetTie-2_SMD_Pad0.5mm, symbol Device:Net-Tie_2
- added G1: EcoTechLogo, Footprints:EcoTech_small, symbol Library:EcoTechLogo
- added RV1: 10k, Potentiometer_THT:Potentiometer_Runtron_RM-065_Vertical, symbol Device:R_POT
Connections:
- net labels added: ADC_POT
- net labels removed: GNDA
- no-connect marks 15 -> 14
Changed lines of the file:
@@
-$EndComp
-$Comp
-L power:GNDA #PWR0117
-U 1 1 5C6A30DC
-P 6350 2650
-F 0 "#PWR0117" H 6350 2400 50  0001 C CNN
-F 1 "GNDA" H 6355 2477 50  0000 C CNN
-F 2 "" H 6350 2650 50  0001 C CNN
-F 3 "" H 6350 2650 50  0001 C CNN
-	1    6350 2650
-	1    0    0    -1
-$EndComp
-$Comp
-L Device:Net-Tie_2 NT1
-U 1 1 5C6A3193
-P 6100 2650
-F 0 "NT1" H 6100 2550 50  0000 C CNN
-F 1 "Net-Tie_2" H 6100 2737 50  0001 C CNN
-F 2 "NetTie:NetTie-2_SMD_Pad0.5mm" H 6100 2650 50  0001 C CNN
-F 3 "~" H 6100 2650 50  0001 C CNN
-	1    6100 2650
-	-1   0    0    -1
-$EndComp
-Wire Wire Line
-	6000 2650 5850 2650
-Wire Wire Line
-	6200 2650 6350 2650
-Connection ~ 6350 2650
-$Comp
-L power:GNDA #PWR0118
-U 1 1 5C6A41FC
-P 9000 3950
-F 0 "#PWR0118" H 9000 3700 50  0001 C CNN
-F 1 "GNDA" H 9100 3800 50  0000 C CNN
-F 2 "" H 9000 3950 50  0001 C CNN
-F 3 "" H 9000 3950 50  0001 C CNN
-	1    9000 3950
-	1    0    0    -1
-$EndComp
-$Comp
-L power:GNDA #PWR0119
-U 1 1 5C6A49D3
-P 8150 2400
-F 0 "#PWR0119" H 8150 2150 50  0001 C CNN
-F 1 "GNDA" H 8155 2227 50  0000 C CNN
-F 2 "" H 8150 2400 50  0001 C CNN
-F 3 "" H 8150 2400 50  0001 C CNN
-	1    8150 2400
-	1    0    0    -1
 $EndComp
 $Comp
@@
 Text Label 2400 6300 0    50   ~ 0
 INLET
-Text Label 1750 7000 2    50   ~ 0
-INLET
 Text Notes 750  6700 1    50   ~ 0
 Wejście sygnału\nzaworu dolotowego
@@
 $EndComp
 Connection ~ 5400 6500
-NoConn ~ 9500 2150
 NoConn ~ 9500 2350
 NoConn ~ 9500 2450
@@
 Wire Wire Line
 	5850 2650 5600 2650
-Connection ~ 5850 2650
 Connection ~ 5600 2650
 Connection ~ 5600 2350
-$Comp
-L power:GNDA #PWR0112
-U 1 1 5CA1826A
-P 9750 2550
-F 0 "#PWR0112" H 9750 2300 50  0001 C CNN
-F 1 "GNDA" H 9850 2400 50  0000 C CNN
-F 2 "" H 9750 2550 50  0001 C CNN
-F 3 "" H 9750 2550 50  0001 C CNN
-	1    9750 2550
-	1    0    0    -1
-$EndComp
 $Comp
 L power:GND #PWR0128
@@
 $EndComp
 Connection ~ 9750 2250
+$Comp
+L Device:R_POT RV1
+U 1 1 5CC5B6AF
+P 10750 3150
+F 0 "RV1" H 10681 3104 50  0000 R CNN
+F 1 "10k" H 10681 3195 50  0000 R CNN
+F 2 "Potentiometer_THT:Potentiometer_Runtron_RM-065_Vertical" H 10750 3150 50  0001 C CNN
+F 3 "~" H 10750 3150 50  0001 C CNN
+	1    10750 3150
+	-1   0    0    1
+$EndComp
+$Comp
+L power:+5VA #PWR0112
+U 1 1 5CC5BA9F
+P 10750 3000
+F 0 "#PWR0112" H 10750 2850 50  0001 C CNN
+F 1 "+5VA" H 10800 3150 50  0000 C CNN
+F 2 "" H 10750 3000 50  0001 C CNN
+F 3 "" H 10750 3000 50  0001 C CNN
+	1    10750 3000
+	1    0    0    -1
+$EndComp
+$Comp
+L power:GND #PWR0117
+U 1 1 5CC5C25C
+P 6350 2650
+F 0 "#PWR0117" H 6350 2400 50  0001 C CNN
+F 1 "GND" H 6355 2477 50  0000 C CNN
+F 2 "" H 6350 2650 50  0001 C CNN
+F 3 "" H 6350 2650 50  0001 C CNN
+	1    6350 2650
+	1    0    0    -1
+$EndComp
+$Comp
+L power:GND #PWR0118
+U 1 1 5CC5C412
+P 8150 2400
+F 0 "#PWR0118" H 8150 2150 50  0001 C CNN
+F 1 "GND" H 8155 2227 50  0000 C CNN
+F 2 "" H 8150 2400 50  0001 C CNN
+F 3 "" H 8150 2400 50  0001 C CNN
+	1    8150 2400
+	1    0    0    -1
+$EndComp
+$Comp
+L power:GND #PWR0119
+U 1 1 5CC5C5C2
+P 9750 2550
+F 0 "#PWR0119" H 9750 2300 50  0001 C CNN
+F 1 "GND" H 9650 2400 50  0000 C CNN
+F 2 "" H 9750 2550 50  0001 C CNN
+F 3 "" H 9750 2550 50  0001 C CNN
+	1    9750 2550
+	-1   0    0    -1
+$EndComp
+$Comp
+L power:GND #PWR0136
+U 1 1 5CC5C772
+P 10750 3300
+F 0 "#PWR0136" H 10750 3050 50  0001 C CNN
+F 1 "GND" H 10650 3150 50  0000 C CNN
+F 2 "" H 10750 3300 50  0001 C CNN
+F 3 "" H 10750 3300 50  0001 C CNN
+	1    10750 3300
+	-1   0    0    -1
+$EndComp
+Wire Wire Line
+	9000 3950 8900 3950
+Connection ~ 8900 3950
+Text Label 9500 2150 0    50   ~ 0
+ADC_POT
+Text Label 10250 3150 0    50   ~ 0
+ADC_POT
+Wire Wire Line
+	10250 3150 10600 3150
+$Comp
+L Library:EcoTechLogo G1
+U 1 1 5CC67452
+P 10600 650
+F 0 "G1" H 10600 750 50  0001 C CNN
+F 1 "EcoTechLogo" H 10625 650 50  0000 L CNN
+F 2 "Footprints:EcoTech_small" H 10600 650 50  0001 C CNN
+F 3 "" H 10600 650 50  0001 C CNN
+	1    10600 650
+	1    0    0    -1
+$EndComp
 $EndSCHEMATC

Commit message: Removed Switches from bus devices and added mounting holes in schematics.
Squashed commit of the following:

commit 448b4f84a5f64686dc4334a0b6d81609891ca7cf
Author: Paweł <mackipawel@gmail.com>
Date:   Sun Apr 28 20:22:14 2019 +0200

    Added mouting holes to SystemSupply.

commit d45917b7024ecbe087cb8328a2c33d3ab10399ff
Author: Paweł <mackipawel@gmail.com>
Date:   Sun Apr 28 20:13:41 2019 +0200

    Added mouting holes to SafetySystem.

commit 6365380671305e2241dc821ec3b00ae08a997ac5
Author: Paweł <mackipawel@gmail.com>
Date:   Sun Apr 28 20:11:13 2019 +0200

    Added mouting holes to SafetySupply.

commit 00163d4bba61eb48f9ebb4c601b04017e78006be
Author: Paweł <mackipawel@gmail.com>
Date:   Sun Apr 28 20:06:38 2019 +0200

    Fixed MotorController.

commit ec0507ca51ef80aebbe2605505e7109beac59e98
Author: Paweł <mackipawel@gmail.com>
Date:   Sun Apr 28 19:54:40 2019 +0200

    Fixed MotorDriver.
Parts:
- added H1, H2, H3, H4: MountingHole, MountingHole:MountingHole_3.2mm_M3, symbol Mechanical:MountingHole
Changed lines of the file:
@@
+	1    0    0    -1
+$EndComp
+$Comp
+L Mechanical:MountingHole H1
+U 1 1 5CC9ACDD
+P 10400 900
+F 0 "H1" H 10500 900 50  0000 L CNN
+F 1 "MountingHole" H 10500 855 50  0001 L CNN
+F 2 "MountingHole:MountingHole_3.2mm_M3" H 10400 900 50  0001 C CNN
+F 3 "~" H 10400 900 50  0001 C CNN
+	1    10400 900
+	1    0    0    -1
+$EndComp
+$Comp
+L Mechanical:MountingHole H2
+U 1 1 5CC9B20D
+P 10700 900
+F 0 "H2" H 10800 900 50  0000 L CNN
+F 1 "MountingHole" H 10800 855 50  0001 L CNN
+F 2 "MountingHole:MountingHole_3.2mm_M3" H 10700 900 50  0001 C CNN
+F 3 "~" H 10700 900 50  0001 C CNN
+	1    10700 900
+	1    0    0    -1
+$EndComp
+$Comp
+L Mechanical:MountingHole H3
+U 1 1 5CC9EB72
+P 10400 1100
+F 0 "H3" H 10500 1100 50  0000 L CNN
+F 1 "MountingHole" H 10500 1055 50  0001 L CNN
+F 2 "MountingHole:MountingHole_3.2mm_M3" H 10400 1100 50  0001 C CNN
+F 3 "~" H 10400 1100 50  0001 C CNN
+	1    10400 1100
+	1    0    0    -1
+$EndComp
+$Comp
+L Mechanical:MountingHole H4
+U 1 1 5CCA24D1
+P 10700 1100
+F 0 "H4" H 10800 1100 50  0000 L CNN
+F 1 "MountingHole" H 10800 1055 50  0001 L CNN
+F 2 "MountingHole:MountingHole_3.2mm_M3" H 10700 1100 50  0001 C CNN
+F 3 "~" H 10700 1100 50  0001 C CNN
+	1    10700 1100
 	1    0    0    -1
 $EndComp
