File: SafetySystem/SafetySystem.sch (KiCad schematic (older format))
At the start: 89 parts, among them J1 Screw_Terminal_01x02, J10 Screw_Terminal_01x02, J2 Screw_Terminal_01x02, J3 Screw_Terminal_01x02, J4 AVR-ISP-10, J5 Screw_Terminal_01x02, J6 Screw_Terminal_01x02, J7 Screw_Terminal_01x02, J8 Screw_Terminal_01x02, J9 Screw_Terminal_01x02, Q1 Q_PMOS_GSD, Q10 Q_NMOS_GSD, Q11 Q_NMOS_GSD, Q12 Q_NMOS_GSD, Q2 Q_PMOS_GSD, Q3 Q_PMOS_GSD, Q4 Q_NMOS_GSD, Q5 Q_NMOS_GSD, Q6 Q_NMOS_GSD, Q7 Q_NMOS_GSD, Q8 Q_NMOS_GSD, Q9 Q_NMOS_GSD, SW2 SW_Push, SW3 SW_Push, SW4 SW_Push, U1 ST1S10PHR, U2 MQ-8, U3 ATmega8A-AU, U4 LTV-817S, U5 LTV-817S, Y1 8Mhz

Commit message: Added testpoints.
Squashed commit of the following:

commit b78741095f1293168643ce5f943c13a7eb09b318
Author: Paweł <mackipawel@gmail.com>
Date:   Thu May 2 10:22:35 2019 +0200

    Added testpoints to remaining projects.

commit d708f3fd02ddff10684a41533d76b9b66ea6c8f4
Author: Paweł <mackipawel@gmail.com>
Date:   Sun Apr 28 23:49:47 2019 +0200

    Added testpoints in MotorController and MotorDriver.
Parts:
- added TP1, TP2, TP3, TP4, TP5, TP6, TP7: TestPoint, TestPoint:TestPoint_Loop_D1.80mm_Drill1.0mm_Beaded, symbol Connector:TestPoint
Connections:
- wire segments 109 -> 112
Changed lines of the file:
@@
 	1    0    0    -1
 $EndComp
-Text Label 3750 2900 0    50   ~ 0
+Text Label 3900 2900 0    50   ~ 0
 SFT_SIG
 $Comp
@@
 U 1 1 5C80277D
 P 4550 6300
-F 0 "R22" V 4650 6200 50  0000 L CNN
+F 0 "R22" V 4650 6150 50  0000 L CNN
 F 1 "2k" V 4650 6350 50  0000 L CNN
 F 2 "Resistor_SMD:R_0603_1608Metric" V 4480 6300 50  0001 C CNN
@@
 U 1 1 5C802784
 P 4700 6450
-F 0 "D12" V 4700 6600 50  0000 R CNN
+F 0 "D12" V 4700 6650 50  0000 R CNN
 F 1 "D_ALT" V 4745 6529 50  0001 L CNN
 F 2 "Diode_SMD:D_MiniMELF" H 4700 6450 50  0001 C CNN
@@
 U 1 1 5C8027A5
 P 6000 6750
-F 0 "D14" V 6000 6900 50  0000 R CNN
+F 0 "D14" V 6000 6950 50  0000 R CNN
 F 1 "D_ALT" V 6045 6829 50  0001 L CNN
 F 2 "Diode_SMD:D_MiniMELF" H 6000 6750 50  0001 C CNN
@@
 U 1 1 5C8027B9
 P 6000 6150
-F 0 "D10" V 6000 6300 50  0000 R CNN
+F 0 "D10" V 6000 6350 50  0000 R CNN
 F 1 "D_ALT" V 6045 6229 50  0001 L CNN
 F 2 "Diode_SMD:D_MiniMELF" H 6000 6150 50  0001 C CNN
@@
 	1    0    0    -1
 $EndComp
+$Comp
+L Connector:TestPoint TP5
+U 1 1 5CCB813C
+P 3650 2900
+F 0 "TP5" H 3708 2974 50  0000 L CNN
+F 1 "TestPoint" H 3708 2929 50  0001 L CNN
+F 2 "TestPoint:TestPoint_Loop_D1.80mm_Drill1.0mm_Beaded" H 3850 2900 50  0001 C CNN
+F 3 "~" H 3850 2900 50  0001 C CNN
+	1    3650 2900
+	1    0    0    -1
+$EndComp
+$Comp
+L Connector:TestPoint TP1
+U 1 1 5CCB863E
+P 3050 1100
+F 0 "TP1" H 3108 1174 50  0000 L CNN
+F 1 "TestPoint" H 3108 1129 50  0001 L CNN
+F 2 "TestPoint:TestPoint_Loop_D1.80mm_Drill1.0mm_Beaded" H 3250 1100 50  0001 C CNN
+F 3 "~" H 3250 1100 50  0001 C CNN
+	1    3050 1100
+	1    0    0    -1
+$EndComp
+$Comp
+L Connector:TestPoint TP3
+U 1 1 5CCBC1A4
+P 3050 1700
+F 0 "TP3" H 3108 1774 50  0000 L CNN
+F 1 "TestPoint" H 3108 1729 50  0001 L CNN
+F 2 "TestPoint:TestPoint_Loop_D1.80mm_Drill1.0mm_Beaded" H 3250 1700 50  0001 C CNN
+F 3 "~" H 3250 1700 50  0001 C CNN
+	1    3050 1700
+	1    0    0    -1
+$EndComp
+$Comp
+L Connector:TestPoint TP4
+U 1 1 5CCC124E
+P 10750 2250
+F 0 "TP4" H 10808 2324 50  0000 L CNN
+F 1 "TestPoint" H 10808 2279 50  0001 L CNN
+F 2 "TestPoint:TestPoint_Loop_D1.80mm_Drill1.0mm_Beaded" H 10950 2250 50  0001 C CNN
+F 3 "~" H 10950 2250 50  0001 C CNN
+	1    10750 2250
+	1    0    0    -1
+$EndComp
+Text Label 10750 2250 2    50   ~ 0
+ADC
+$Comp
+L Connector:TestPoint TP2
+U 1 1 5CCC1946
+P 6600 1100
+F 0 "TP2" H 6658 1174 50  0000 L CNN
+F 1 "TestPoint" H 6658 1129 50  0001 L CNN
+F 2 "TestPoint:TestPoint_Loop_D1.80mm_Drill1.0mm_Beaded" H 6800 1100 50  0001 C CNN
+F 3 "~" H 6800 1100 50  0001 C CNN
+	1    6600 1100
+	1    0    0    -1
+$EndComp
+Wire Wire Line
+	6600 1100 6400 1100
+Wire Wire Line
+	3050 1100 2600 1100
+Wire Wire Line
+	3050 1700 2600 1700
+Connection ~ 2600 1700
+$Comp
+L Connector:TestPoint TP6
+U 1 1 5CCD1351
+P 5400 6500
+F 0 "TP6" H 5400 6700 50  0000 L CNN
+F 1 "TestPoint" H 5458 6529 50  0001 L CNN
+F 2 "TestPoint:TestPoint_Loop_D1.80mm_Drill1.0mm_Beaded" H 5600 6500 50  0001 C CNN
+F 3 "~" H 5600 6500 50  0001 C CNN
+	1    5400 6500
+	1    0    0    -1
+$EndComp
+$Comp
+L Connector:TestPoint TP7
+U 1 1 5CCD51E7
+P 2100 6500
+F 0 "TP7" H 2150 6700 50  0000 L CNN
+F 1 "TestPoint" H 2158 6529 50  0001 L CNN
+F 2 "TestPoint:TestPoint_Loop_D1.80mm_Drill1.0mm_Beaded" H 2300 6500 50  0001 C CNN
+F 3 "~" H 2300 6500 50  0001 C CNN
+	1    2100 6500
+	1    0    0    -1
+$EndComp

Commit message: Added 3D models to the library
Squashed commit of the following:

commit 8070c09fc3d8f70a7cb84d0f12b6782c2c87c14c
Author: Paweł <mackipawel@gmail.com>
Date:   Mon May 6 20:26:56 2019 +0200

    Added SystemSupply 3d models.

commit 94ef8708632c7bc91211bc6ded4e0c8fb9ccef4a
Author: Paweł <mackipawel@gmail.com>
Date:   Mon May 6 01:08:52 2019 +0200

    Added 3D models to SystemSupply.

commit eb394d70be979be958e4acab21accb1817e8e0e5
Author: Paweł <mackipawel@gmail.com>
Date:   Mon May 6 00:55:39 2019 +0200

    Added 3D model to MotorController.

commit fd89e01e0ef36f85afad3e8686d3deffdf36454d
Author: Paweł <mackipawel@gmail.com>
Date:   Mon May 6 00:40:56 2019 +0200

    Added 3D models in MotorDriver.

commit 899d106fa8d45578189a4955328047d8f9558beb
Author: Paweł <mackipawel@gmail.com>
Date:   Mon May 6 00:09:40 2019 +0200

    Added 3D models to SafetySupply.

commit 06c807994bb47431d2802a96796741a0e8fb9ae5
Author: Paweł <mackipawel@gmail.com>
Date:   Sun May 5 23:17:48 2019 +0200

    Added 3D models to SafetySystem.
Parts:
- RV1: footprint Potentiometer_THT:Potentiometer_Runtron_RM-065_Vertical -> Footprints:Potentiometer_Runtron_RM-065_Vertical
- SW3, SW4: footprint Button_Switch_THT:SW_PUSH-12mm -> Footprints:SW_PUSH-12mm
- Y1: footprint Crystal:Crystal_SMD_HC49-SD -> Footprints:Crystal_SMD_HC49-SD
Changed lines of the file:
@@
 F 0 "SW3" H 3450 3100 50  0000 C CNN
 F 1 "SW_Push" H 3450 3394 50  0001 C CNN
-F 2 "Button_Switch_THT:SW_PUSH-12mm" H 3450 3400 50  0001 C CNN
+F 2 "Footprints:SW_PUSH-12mm" H 3450 3400 50  0001 C CNN
 F 3 "" H 3450 3400 50  0001 C CNN
 	1    3450 3200
@@
 F 0 "SW4" V 2700 6500 50  0000 C CNN
 F 1 "SW_Push" H 2700 6794 50  0001 C CNN
-F 2 "Button_Switch_THT:SW_PUSH-12mm" H 2700 6800 50  0001 C CNN
+F 2 "Footprints:SW_PUSH-12mm" H 2700 6800 50  0001 C CNN
 F 3 "" H 2700 6800 50  0001 C CNN
 	1    2700 6600
@@
 F 0 "Y1" H 7300 1900 50  0000 C CNN
 F 1 "8Mhz" H 7250 1800 50  0000 C CNN
-F 2 "Crystal:Crystal_SMD_HC49-SD" H 7550 1850 50  0001 C CNN
+F 2 "Footprints:Crystal_SMD_HC49-SD" H 7550 1850 50  0001 C CNN
 F 3 "~" H 7550 1850 50  0001 C CNN
 	1    7550 1850
@@
 F 0 "RV1" H 10681 3104 50  0000 R CNN
 F 1 "10k" H 10681 3195 50  0000 R CNN
-F 2 "Potentiometer_THT:Potentiometer_Runtron_RM-065_Vertical" H 10750 3150 50  0001 C CNN
+F 2 "Footprints:Potentiometer_Runtron_RM-065_Vertical" H 10750 3150 50  0001 C CNN
 F 3 "~" H 10750 3150 50  0001 C CNN
 	1    10750 3150
