File: SystemSupply/SystemSupply.sch (KiCad schematic (older format))
At the start: 44 parts, among them J1 Conn_01x01, J10 Screw_Terminal_01x02, J2 Conn_01x01, J3 4P4C, J4 Conn_01x01, J5 Conn_01x01, J6 Screw_Terminal_01x02, J7 4P4C, J8 Screw_Terminal_01x02, J9 Screw_Terminal_01x02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

Commit message: System supply PCB
Squashed commit of the following:

commit dbc07ea87a8cb2914ffd081ab2f264bc75cd574d
Author: Paweł <mackipawel@gmail.com>
Date:   Wed Apr 10 22:15:52 2019 +0200

    Added polygon pours and edited silk screen designators.

commit e8e96d6977d739eab19b0dc30615939eafea5188
Author: Paweł <mackipawel@gmail.com>
Date:   Wed Apr 10 21:41:22 2019 +0200

    Routed tracks.

commit 0491c31da248ed480bc4eeb27d8c4f7c530a2869
Author: Paweł <mackipawel@gmail.com>
Date:   Wed Apr 10 00:03:41 2019 +0200

    Placed elements on PCB.
Parts:
- removed D4: D_TVS_ALT, Diode_SMD:D_SMC, symbol Device:D_TVS_ALT
- added JP5: Jumper_NO_Small, Jumper:SolderJumper-2_P1.3mm_Open_TrianglePad1.0x1.5mm, symbol Device:Jumper_NO_Small
- C2: footprint Capacitor_SMD:C_0603_1608Metric -> Capacitor_SMD:C_0805_2012Metric
- C3, C4: footprint Capacitor_THT:C_Radial_D10.0mm_H20.0mm_P5.00mm -> Footprints:C_Radial_D6.3mm_H11.0mm_P2.50mm
- SW1, SW2: footprint Footprints:5MS1S102AM6QE -> Footprints:5MS1S102AM2QE
Connections:
- wire segments 97 -> 100
Other:
- moved on the sheet: D2, D5, J8
Changed lines of the file:
@@
 L power:GND #PWR06
 U 1 1 5C72F659
-P 8550 1800
-F 0 "#PWR06" H 8550 1550 50  0001 C CNN
-F 1 "GND" H 8555 1627 50  0000 C CNN
-F 2 "" H 8550 1800 50  0001 C CNN
-F 3 "" H 8550 1800 50  0001 C CNN
-	1    8550 1800
+P 8550 1850
+F 0 "#PWR06" H 8550 1600 50  0001 C CNN
+F 1 "GND" H 8555 1677 50  0000 C CNN
+F 2 "" H 8550 1850 50  0001 C CNN
+F 3 "" H 8550 1850 50  0001 C CNN
+	1    8550 1850
 	1    0    0    -1
 $EndComp
@@
 Wire Wire Line
 	8550 1700 9100 1700
-Wire Wire Line
-	8550 1800 8550 1700
 Text Notes 8050 1000 0    50   ~ 0
 Włącznik zasilania magistrali
@@
 L power:+12V #PWR012
 U 1 1 5C753CF7
-P 4900 3250
-F 0 "#PWR012" H 4900 3100 50  0001 C CNN
-F 1 "+12V" H 4915 3423 50  0000 C CNN
-F 2 "" H 4900 3250 50  0001 C CNN
-F 3 "" H 4900 3250 50  0001 C CNN
-	1    4900 3250
+P 4900 3100
+F 0 "#PWR012" H 4900 2950 50  0001 C CNN
+F 1 "+12V" H 4915 3273 50  0000 C CNN
+F 2 "" H 4900 3100 50  0001 C CNN
+F 3 "" H 4900 3100 50  0001 C CNN
+	1    4900 3100
 	1    0    0    -1
 $EndComp
@@
 Podły chińczyk
 $Comp
-L Device:D_TVS_ALT D4
-U 1 1 5C75BDAE
-P 2400 3400
-F 0 "D4" V 2400 3479 50  0000 L CNN
-F 1 "D_TVS_ALT" V 2445 3479 50  0001 L CNN
-F 2 "Diode_SMD:D_SMC" H 2400 3400 50  0001 C CNN
-F 3 "" H 2400 3400 50  0001 C CNN
-	1    2400 3400
-	0    1    1    0
-$EndComp
-$Comp
 L power:+24V #PWR011
 U 1 1 5C75BE3F
@@
 F 0 "C2" H 2815 3446 50  0000 L CNN
 F 1 "10n" H 2815 3355 50  0000 L CNN
-F 2 "Capacitor_SMD:C_0603_1608Metric" H 2738 3250 50  0001 C CNN
+F 2 "Capacitor_SMD:C_0805_2012Metric" H 2738 3250 50  0001 C CNN
 F 3 "~" H 2700 3400 50  0001 C CNN
 F 4 "X1" H 2700 3400 50  0001 C CNN "Type"
@@
 	2700 3250 2400 3250
 Connection ~ 2400 3250
-Wire Wire Line
-	1900 3550 2400 3550
-Connection ~ 2400 3550
 $Comp
 L Device:CP C3
@@
 F 0 "C3" H 3368 3446 50  0000 L CNN
 F 1 "470u" H 3368 3355 50  0000 L CNN
-F 2 "Capacitor_THT:C_Radial_D10.0mm_H20.0mm_P5.00mm" H 3288 3250 50  0001 C CNN
+F 2 "Footprints:C_Radial_D6.3mm_H11.0mm_P2.50mm" H 3288 3250 50  0001 C CNN
 F 3 "~" H 3250 3400 50  0001 C CNN
 F 4 "50V" H 3250 3400 50  0001 C CNN "Voltage"
@@
 L Connector:Screw_Terminal_01x02 J8
 U 1 1 5C78DF54
-P 9700 4100
-F 0 "J8" H 9619 3867 50  0000 C CNN
-F 1 "Screw_Terminal_01x02" H 9620 3866 50  0001 C CNN
-F 2 "Footprints:TerminalBlock_DG250_02P" H 9700 4100 50  0001 C CNN
-F 3 "" H 9700 4100 50  0001 C CNN
-	1    9700 4100
+P 9750 4350
+F 0 "J8" H 9669 4117 50  0000 C CNN
+F 1 "Screw_Terminal_01x02" H 9670 4116 50  0001 C CNN
+F 2 "Footprints:TerminalBlock_DG250_02P" H 9750 4350 50  0001 C CNN
+F 3 "" H 9750 4350 50  0001 C CNN
+	1    9750 4350
 	1    0    0    1
 $EndComp
@@
 L power:GND #PWR016
 U 1 1 5C78E1E1
-P 9100 4100
-F 0 "#PWR016" H 9100 3850 50  0001 C CNN
-F 1 "GND" H 9105 3927 50  0000 C CNN
-F 2 "" H 9100 4100 50  0001 C CNN
-F 3 "" H 9100 4100 50  0001 C CNN
-	1    9100 4100
-	1    0    0    -1
-$EndComp
-Wire Wire Line
-	9100 4100 9500 4100
-Text Notes 9050 3450 0    50   ~ 0
+P 9400 4550
+F 0 "#PWR016" H 9400 4300 50  0001 C CNN
+F 1 "GND" H 9405 4377 50  0000 C CNN
+F 2 "" H 9400 4550 50  0001 C CNN
+F 3 "" H 9400 4550 50  0001 C CNN
+	1    9400 4550
+	1    0    0    -1
+$EndComp
+Text Notes 9200 3750 0    50   ~ 0
 Zasilanie sterownika ogniwa
 $Comp
@@
 F 0 "C4" H 5018 3446 50  0000 L CNN
 F 1 "180u" H 5018 3355 50  0000 L CNN
-F 2 "Capacitor_THT:C_Radial_D10.0mm_H20.0mm_P5.00mm" H 4938 3250 50  0001 C CNN
+F 2 "Footprints:C_Radial_D6.3mm_H11.0mm_P2.50mm" H 4938 3250 50  0001 C CNN
 F 3 "~" H 4900 3400 50  0001 C CNN
 F 4 "50V" H 4900 3400 50  0001 C CNN "Voltage"
@@
 	1    0    0    -1
 $EndComp
-Connection ~ 4900 3250
 Connection ~ 4900 3550
 Wire Wire Line
@@
 U 1 1 5C77DEF5
 P 4650 3250
-F 0 "L2" V 4840 3250 50  0000 C CNN
-F 1 "3u" V 4749 3250 50  0000 C CNN
+F 0 "L2" V 4550 3150 50  0000 C CNN
+F 1 "3u" V 4550 3300 50  0000 C CNN
 F 2 "Inductor_SMD:L_1812_4532Metric" H 4650 3250 50  0001 C CNN
 F 3 "~" H 4650 3250 50  0001 C CNN
 F 4 "2A" V 4650 3250 50  0001 C CNN "Current"
 	1    4650 3250
-	0    -1   -1   0
+	0    1    -1   0
 $EndComp
 $Comp
@@
 Przemysłowy pewniak
 Wire Wire Line
-	2400 3550 2700 3550
-Wire Wire Line
 	2400 3250 2350 3250
 Wire Wire Line
@@
 L Switch:SW_SPDT SW1
 U 1 1 5CA35DAC
-P 8750 1500
-F 0 "SW1" H 8750 1693 50  0000 C CNN
-F 1 "SW_SPDT" H 8750 1694 50  0001 C CNN
-F 2 "Footprints:5MS1S102AM6QE" H 8750 1500 50  0001 C CNN
-F 3 "" H 8750 1500 50  0001 C CNN
-	1    8750 1500
-	1    0    0    -1
-$EndComp
-Connection ~ 8950 1600
-Wire Wire Line
-	8950 1400 8950 1350
-Wire Wire Line
-	8950 1350 8550 1350
-Connection ~ 8550 1350
-Wire Wire Line
-	8550 1350 8550 1500
+P 8750 1450
+F 0 "SW1" H 8750 1643 50  0000 C CNN
+F 1 "SW_SPDT" H 8750 1644 50  0001 C CNN
+F 2 "Footprints:5MS1S102AM2QE" H 8750 1450 50  0001 C CNN
+F 3 "" H 8750 1450 50  0001 C CNN
+	1    8750 1450
+	-1   0    0    -1
+$EndComp
 $Comp
 L Library:R30N K1
@@
 F 3 "https://www.tme.eu/pl/Document/d84e58b273b47d235ca1e19ed7eca28c/R30N-PL.pdf" H 2100 1650 50  0001 C CNN
 	1    2100 1650
-	0    1    -1   0
+	0    -1   -1   0
 $EndComp
 $Comp
 L power:+12V #PWR015
 U 1 1 5CA3EC14
-P 9100 3750
-F 0 "#PWR015" H 9100 3600 50  0001 C CNN
-F 1 "+12V" H 9115 3923 50  0000 C CNN
-F 2 "" H 9100 3750 50  0001 C CNN
-F 3 "" H 9100 3750 50  0001 C CNN
-	1    9100 3750
+P 8950 4000
+F 0 "#PWR015" H 8950 3850 50  0001 C CNN
+F 1 "+12V" H 8965 4173 50  0000 C CNN
+F 2 "" H 8950 4000 50  0001 C CNN
+F 3 "" H 8950 4000 50  0001 C CNN
+	1    8950 4000
 	1    0    0    -1
 $EndComp
@@
 L Switch:SW_SPDT SW2
 U 1 1 5CA3EC1A
-P 9300 3900
-F 0 "SW2" H 9300 4093 50  0000 C CNN
-F 1 "SW_SPDT" H 9300 4094 50  0001 C CNN
-F 2 "Footprints:5MS1S102AM6QE" H 9300 3900 50  0001 C CNN
-F 3 "" H 9300 3900 50  0001 C CNN
-	1    9300 3900
-	1    0    0    -1
-$EndComp
-Wire Wire Line
-	9500 3750 9100 3750
-Connection ~ 9100 3750
-Wire Wire Line
-	9100 3750 9100 3900
-Wire Wire Line
-	9500 3800 9500 3750
+P 9200 4100
+F 0 "SW2" H 9200 4293 50  0000 C CNN
+F 1 "SW_SPDT" H 9200 4294 50  0001 C CNN
+F 2 "Footprints:5MS1S102AM2QE" H 9200 4100 50  0001 C CNN
+F 3 "" H 9200 4100 50  0001 C CNN
+	1    9200 4100
+	-1   0    0    -1
+$EndComp
 $Comp
 L Device:D_TVS_ALT D5
 U 1 1 5CA494E3
-P 9000 3950
-F 0 "D5" V 9000 4029 50  0000 L CNN
-F 1 "D_TVS_ALT" V 9045 4029 50  0001 L CNN
-F 2 "Diode_SMD:D_SMC" H 9000 3950 50  0001 C CNN
-F 3 "" H 9000 3950 50  0001 C CNN
-	1    9000 3950
+P 9400 4400
+F 0 "D5" V 9400 4479 50  0000 L CNN
+F 1 "D_TVS_ALT" V 9445 4479 50  0001 L CNN
+F 2 "Diode_SMD:D_SMC" H 9400 4400 50  0001 C CNN
+F 3 "" H 9400 4400 50  0001 C CNN
+	1    9400 4400
 	0    -1   1    0
 $EndComp
-Wire Wire Line
-	9000 4100 9100 4100
-Connection ~ 9100 4100
-Wire Wire Line
-	9000 3800 9000 3750
-Wire Wire Line
-	9000 3750 9100 3750
 $Comp
 L Device:D_TVS_ALT D2
 U 1 1 5CA50CD4
-P 8400 1600
-F 0 "D2" V 8400 1679 50  0000 L CNN
-F 1 "D_TVS_ALT" V 8445 1679 50  0001 L CNN
-F 2 "Diode_SMD:D_SMC" H 8400 1600 50  0001 C CNN
-F 3 "" H 8400 1600 50  0001 C CNN
-	1    8400 1600
+P 8400 1700
+F 0 "D2" V 8400 1779 50  0000 L CNN
+F 1 "D_TVS_ALT" V 8445 1779 50  0001 L CNN
+F 2 "Diode_SMD:D_SMC" H 8400 1700 50  0001 C CNN
+F 3 "" H 8400 1700 50  0001 C CNN
+	1    8400 1700
 	0    -1   1    0
 $EndComp
 Wire Wire Line
-	8400 1450 8400 1350
-Wire Wire Line
-	8400 1350 8550 1350
-Wire Wire Line
-	8400 1750 8400 1800
-Wire Wire Line
-	8400 1800 8550 1800
-Connection ~ 8550 1800
+	8400 1850 8550 1850
+Connection ~ 8550 1850
+Wire Wire Line
+	2400 1350 2400 1450
+Wire Wire Line
+	1800 1450 1800 1350
+Wire Wire Line
+	1900 3550 2700 3550
+Wire Wire Line
+	8950 1450 8950 1600
+Connection ~ 8950 1600
+Wire Wire Line
+	8550 1600 8950 1600
+Wire Wire Line
+	8550 1550 8400 1550
+Connection ~ 8550 1550
+Wire Wire Line
+	8550 1550 8550 1600
+Wire Wire Line
+	8550 1700 8550 1850
+Wire Wire Line
+	9000 4200 9000 4250
+Wire Wire Line
+	9000 4250 9400 4250
+Wire Wire Line
+	9400 4250 9400 4100
+Connection ~ 9400 4250
+Wire Wire Line
+	9550 4350 9550 4550
+Wire Wire Line
+	9550 4550 9400 4550
+Connection ~ 9400 4550
+Wire Wire Line
+	9550 4250 9400 4250
+Wire Wire Line
+	8950 4000 9000 4000
+$Comp
+L Device:Jumper_NO_Small JP5
+U 1 1 5CAE5906
+P 4650 3100
+F 0 "JP5" H 4650 3193 50  0000 C CNN
+F 1 "Jumper_NO_Small" H 4650 3194 50  0001 C CNN
+F 2 "Jumper:SolderJumper-2_P1.3mm_Open_TrianglePad1.0x1.5mm" H 4650 3100 50  0001 C CNN
+F 3 "~" H 4650 3100 50  0001 C CNN
+	1    4650 3100
+	1    0    0    -1
+$EndComp
+Connection ~ 4900 3250
+Wire Wire Line
+	4750 3100 4900 3100
+Wire Wire Line
+	4900 3100 4900 3250
+Connection ~ 4900 3100
+Wire Wire Line
+	4550 3100 4500 3100
+Wire Wire Line
+	4500 3100 4500 3250
+Connection ~ 4500 3250
 $EndSCHEMATC

Commit message: Removed Switches from bus devices and added mounting holes in schematics.
Squashed commit of the following:

commit 448b4f84a5f64686dc4334a0b6d81609891ca7cf
Author: Paweł <mackipawel@gmail.com>
Date:   Sun Apr 28 20:22:14 2019 +0200

    Added mouting holes to SystemSupply.

commit d45917b7024ecbe087cb8328a2c33d3ab10399ff
Author: Paweł <mackipawel@gmail.com>
Date:   Sun Apr 28 20:13:41 2019 +0200

    Added mouting holes to SafetySystem.

commit 6365380671305e2241dc821ec3b00ae08a997ac5
Author: Paweł <mackipawel@gmail.com>
Date:   Sun Apr 28 20:11:13 2019 +0200

    Added mouting holes to SafetySupply.

commit 00163d4bba61eb48f9ebb4c601b04017e78006be
Author: Paweł <mackipawel@gmail.com>
Date:   Sun Apr 28 20:06:38 2019 +0200

    Fixed MotorController.

commit ec0507ca51ef80aebbe2605505e7109beac59e98
Author: Paweł <mackipawel@gmail.com>
Date:   Sun Apr 28 19:54:40 2019 +0200

    Fixed MotorDriver.
Parts:
- added G1: EcoTechLogo, Footprints:EcoTech, symbol Library:EcoTechLogo
- added H1, H2, H3, H4: MountingHole, MountingHole:MountingHole_3.2mm_M3, symbol Mechanical:MountingHole
Changed lines of the file:
@@
 	4500 3100 4500 3250
 Connection ~ 4500 3250
+$Comp
+L Mechanical:MountingHole H1
+U 1 1 5CCA9CDE
+P 6050 1150
+F 0 "H1" H 6150 1150 50  0000 L CNN
+F 1 "MountingHole" H 6150 1105 50  0001 L CNN
+F 2 "MountingHole:MountingHole_3.2mm_M3" H 6050 1150 50  0001 C CNN
+F 3 "~" H 6050 1150 50  0001 C CNN
+	1    6050 1150
+	1    0    0    -1
+$EndComp
+$Comp
+L Mechanical:MountingHole H2
+U 1 1 5CCA9EC4
+P 6350 1150
+F 0 "H2" H 6450 1150 50  0000 L CNN
+F 1 "MountingHole" H 6450 1105 50  0001 L CNN
+F 2 "MountingHole:MountingHole_3.2mm_M3" H 6350 1150 50  0001 C CNN
+F 3 "~" H 6350 1150 50  0001 C CNN
+	1    6350 1150
+	1    0    0    -1
+$EndComp
+$Comp
+L Mechanical:MountingHole H3
+U 1 1 5CCACC01
+P 6050 1350
+F 0 "H3" H 6150 1350 50  0000 L CNN
+F 1 "MountingHole" H 6150 1305 50  0001 L CNN
+F 2 "MountingHole:MountingHole_3.2mm_M3" H 6050 1350 50  0001 C CNN
+F 3 "~" H 6050 1350 50  0001 C CNN
+	1    6050 1350
+	1    0    0    -1
+$EndComp
+$Comp
+L Mechanical:MountingHole H4
+U 1 1 5CCAF938
+P 6350 1350
+F 0 "H4" H 6450 1350 50  0000 L CNN
+F 1 "MountingHole" H 6450 1305 50  0001 L CNN
+F 2 "MountingHole:MountingHole_3.2mm_M3" H 6350 1350 50  0001 C CNN
+F 3 "~" H 6350 1350 50  0001 C CNN
+	1    6350 1350
+	1    0    0    -1
+$EndComp
+$Comp
+L Library:EcoTechLogo G1
+U 1 1 5CCB2A30
+P 6000 950
+F 0 "G1" H 6000 1050 50  0001 C CNN
+F 1 "EcoTechLogo" H 6025 950 50  0000 L CNN
+F 2 "Footprints:EcoTech" H 6000 950 50  0001 C CNN
+F 3 "" H 6000 950 50  0001 C CNN
+	1    6000 950
+	1    0    0    -1
+$EndComp
 $EndSCHEMATC

Commit message: Added testpoints.
Squashed commit of the following:

commit b78741095f1293168643ce5f943c13a7eb09b318
Author: Paweł <mackipawel@gmail.com>
Date:   Thu May 2 10:22:35 2019 +0200

    Added testpoints to remaining projects.

commit d708f3fd02ddff10684a41533d76b9b66ea6c8f4
Author: Paweł <mackipawel@gmail.com>
Date:   Sun Apr 28 23:49:47 2019 +0200

    Added testpoints in MotorController and MotorDriver.
Parts:
- added TP1, TP5, TP6: TestPoint, TestPoint:TestPoint_Loop_D1.80mm_Drill1.0mm_Beaded, symbol Connector:TestPoint
Connections:
- wire segments 100 -> 102
Changed lines of the file:
@@
 U 1 1 5C792763
 P 4900 3400
-F 0 "C4" H 5018 3446 50  0000 L CNN
-F 1 "180u" H 5018 3355 50  0000 L CNN
+F 0 "C4" H 5050 3500 50  0000 L CNN
+F 1 "180u" H 4650 3300 50  0000 L CNN
 F 2 "Footprints:C_Radial_D6.3mm_H11.0mm_P2.50mm" H 4938 3250 50  0001 C CNN
 F 3 "~" H 4900 3400 50  0001 C CNN
@@
 	1    0    0    -1
 $EndComp
+$Comp
+L Connector:TestPoint TP1
+U 1 1 5CCDEDD3
+P 2900 1350
+F 0 "TP1" H 2958 1424 50  0000 L CNN
+F 1 "TestPoint" H 2958 1379 50  0001 L CNN
+F 2 "TestPoint:TestPoint_Loop_D1.80mm_Drill1.0mm_Beaded" H 3100 1350 50  0001 C CNN
+F 3 "~" H 3100 1350 50  0001 C CNN
+	1    2900 1350
+	1    0    0    -1
+$EndComp
+$Comp
+L Connector:TestPoint TP5
+U 1 1 5CCDF736
+P 5100 3100
+F 0 "TP5" H 5158 3174 50  0000 L CNN
+F 1 "TestPoint" H 5158 3129 50  0001 L CNN
+F 2 "TestPoint:TestPoint_Loop_D1.80mm_Drill1.0mm_Beaded" H 5300 3100 50  0001 C CNN
+F 3 "~" H 5300 3100 50  0001 C CNN
+	1    5100 3100
+	1    0    0    -1
+$EndComp
+$Comp
+L Connector:TestPoint TP6
+U 1 1 5CCDF819
+P 5100 3550
+F 0 "TP6" H 5158 3624 50  0000 L CNN
+F 1 "TestPoint" H 5158 3579 50  0001 L CNN
+F 2 "TestPoint:TestPoint_Loop_D1.80mm_Drill1.0mm_Beaded" H 5300 3550 50  0001 C CNN
+F 3 "~" H 5300 3550 50  0001 C CNN
+	1    5100 3550
+	1    0    0    -1
+$EndComp
+Wire Wire Line
+	5100 3550 4900 3550
+Wire Wire Line
+	5100 3100 4900 3100
 $EndSCHEMATC

Commit message: Added 3D models to the library
Squashed commit of the following:

commit 8070c09fc3d8f70a7cb84d0f12b6782c2c87c14c
Author: Paweł <mackipawel@gmail.com>
Date:   Mon May 6 20:26:56 2019 +0200

    Added SystemSupply 3d models.

commit 94ef8708632c7bc91211bc6ded4e0c8fb9ccef4a
Author: Paweł <mackipawel@gmail.com>
Date:   Mon May 6 01:08:52 2019 +0200

    Added 3D models to SystemSupply.

commit eb394d70be979be958e4acab21accb1817e8e0e5
Author: Paweł <mackipawel@gmail.com>
Date:   Mon May 6 00:55:39 2019 +0200

    Added 3D model to MotorController.

commit fd89e01e0ef36f85afad3e8686d3deffdf36454d
Author: Paweł <mackipawel@gmail.com>
Date:   Mon May 6 00:40:56 2019 +0200

    Added 3D models in MotorDriver.

commit 899d106fa8d45578189a4955328047d8f9558beb
Author: Paweł <mackipawel@gmail.com>
Date:   Mon May 6 00:09:40 2019 +0200

    Added 3D models to SafetySupply.

commit 06c807994bb47431d2802a96796741a0e8fb9ae5
Author: Paweł <mackipawel@gmail.com>
Date:   Sun May 5 23:17:48 2019 +0200

    Added 3D models to SafetySystem.
Parts:
- C3, C4: footprint Footprints:C_Radial_D6.3mm_H11.0mm_P2.50mm -> Footprints:C_Radial_D5.0mm_H11.0mm_P2.00mm
- SW3: footprint Button_Switch_THT:SW_PUSH-12mm -> Footprints:SW_PUSH-12mm
Changed lines of the file:
@@
 F 0 "SW3" V 3800 6998 50  0000 L CNN
 F 1 "SW_Push" V 3845 6998 50  0001 L CNN
-F 2 "Button_Switch_THT:SW_PUSH-12mm" H 3800 7050 50  0001 C CNN
+F 2 "Footprints:SW_PUSH-12mm" H 3800 7050 50  0001 C CNN
 F 3 "" H 3800 7050 50  0001 C CNN
 	1    3800 6850
@@
 F 0 "C3" H 3368 3446 50  0000 L CNN
 F 1 "470u" H 3368 3355 50  0000 L CNN
-F 2 "Footprints:C_Radial_D6.3mm_H11.0mm_P2.50mm" H 3288 3250 50  0001 C CNN
+F 2 "Footprints:C_Radial_D5.0mm_H11.0mm_P2.00mm" H 3288 3250 50  0001 C CNN
 F 3 "~" H 3250 3400 50  0001 C CNN
 F 4 "50V" H 3250 3400 50  0001 C CNN "Voltage"
@@
 F 0 "C4" H 5050 3500 50  0000 L CNN
 F 1 "180u" H 4650 3300 50  0000 L CNN
-F 2 "Footprints:C_Radial_D6.3mm_H11.0mm_P2.50mm" H 4938 3250 50  0001 C CNN
+F 2 "Footprints:C_Radial_D5.0mm_H11.0mm_P2.00mm" H 4938 3250 50  0001 C CNN
 F 3 "~" H 4900 3400 50  0001 C CNN
 F 4 "50V" H 4900 3400 50  0001 C CNN "Voltage"
