File: Telemetry/Telemetry_v1.0.1.kicad_pcb (KiCad board)
At the start: 2 copper layers, 56.5 x 55 mm, 60 parts, among them J1 Micro_SD_Card, J5 Conn_02x05_Odd_Even, J7 4P4C, J8 4P4C, Q3 Q_NMOS_GSD, SW1 SW_Push, SW3 SW_Push, U3 MAX485E, U4 STM32F103C8Tx, U5 LD1117S50TR_SOT223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

Commit message: create version 1.0.1
Signed-off-by: Cezary Sobczak <cezary.sobczak@3mdeb.com>
Parts:
- moved D9 10.3 mm to (139.0, 113.2), turned to 180 degrees
- moved D5 6.90 mm to (121.0, 142.8)
- moved R11 6.90 mm to (121.0, 139.1)
- moved D7 6.80 mm to (127.8, 142.7)
- moved R13 6.80 mm to (127.8, 139.1)
- moved R10 0.70 mm to (147.5, 146.0), turned to 0 degrees
- moved D6 0.22 mm to (124.4, 142.7)
- moved R12 0.22 mm to (124.4, 139.1)
- turned C10 to 0 degrees
Connections:
- JP4 pad : /4 -> (no net)
- JP5 pad : Net-(J5-Pad5) -> (no net)
- JP6 pad : /2 -> (no net)
Routing:
- net +3V3: track 121.0 -> 0.01 mm, vias 1 -> 0
- net +12V: track 74.5 -> 0.00 mm
- net Net-(SW3-Pad1): track 51.3 -> 0.00 mm
- net /A: track 44.3 -> 0.00 mm, vias 1 -> 0
- net +5V: track 40.5 -> 0.00 mm
- net /B: track 40.4 -> 0.00 mm, vias 1 -> 0
- net /RST: track 35.7 -> 0.00 mm, vias 2 -> 0
- net /2: track 28.3 -> 0.00 mm
- net /MOSI: track 25.6 -> 0.00 mm
- net /SCK: track 24.7 -> 0.00 mm
- net Net-(C11-Pad1): track 20.6 -> 0.00 mm, vias 2 -> 0
- net /CS: track 20.3 -> 0.00 mm, vias 2 -> 0
- net /MISO: track 19.0 -> 0.00 mm
- net /RX: track 17.5 -> 0.00 mm, vias 2 -> 0
- net /LED1: track 16.7 -> 0.00 mm, vias 2 -> 0
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